File: hardware/pcb/eagle/front_end_block.brd (EAGLE design)
At the start: 30 x 25 mm, 29 parts, among them T1 DDTC114, T2 DDTC114, U1 MAX2769LPKF, X1 SMA

Commit message: Getting libraries to work...
Routing:
- net GNDA: track 61.5 -> 64.5 mm
Changed lines of the file:
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@@
 <wire x1="23.25" y1="17.5" x2="23.25" y2="16.05" width="0.6096" layer="1"/>
 <polygon width="0.254" layer="16">
-<vertex x="0" y="0"/>
+<vertex x="2" y="0"/>
 <vertex x="30" y="0"/>
 <vertex x="30" y="25"/>
-<vertex x="0" y="25"/>
+<vertex x="2" y="25"/>
 </polygon>
 <via x="5" y="0" extent="1-16" drill="1.3" diameter="1.9304"/>
@@
 <wire x1="15.45" y1="21.5" x2="15.55" y2="21.4" width="0.3048" layer="1"/>
 <wire x1="9.9" y1="6.8" x2="9.9" y2="7.6" width="0.3048" layer="1"/>
+<wire x1="0" y1="15" x2="3" y2="15" width="2.1844" layer="16"/>
 </signal>
 <signal name="XTAL">
