File: hardware/pcb/kicad/base_station_clock.sch (KiCad schematic (older format))
At the start: 8 parts, among them U2 XTAL_DRIVER, X1 TCXO

Commit message: Getting libraries to work...
Parts:
- removed U2: XTAL_DRIVER, MODULE, symbol XTAL_DRIVER
- removed X1: TCXO, MODULE, symbol TCXO
- added U2: XTAL_DRIVER_TART, MODULE, symbol XTAL_DRIVER_TART
- added X1: TCXO_TART, MODULE, symbol TCXO_TART
- renumbered C21 to C26, C22 to C27, R29 to R30, R30 to R31, R31 to R32, R32 to R33
Changed lines of the file:
@@
-EESchema Schematic File Version 2  date Tue 09 Sep 2014 11:32:54 NZST
+EESchema Schematic File Version 2  date Wed 17 Sep 2014 15:47:12 NZST
 LIBS:power
 LIBS:device
@@
 LIBS:valves
 LIBS:TART
-LIBS:Papilio
 LIBS:base_station_integrated-cache
 EELAYER 25  0
@@
 $Descr A4 11700 8267
 encoding utf-8
-Sheet 6 7
+Sheet 7 7
 Title ""
-Date "8 sep 2014"
+Date "17 sep 2014"
 Rev ""
 Comp ""
@@
 $EndDescr
 $Comp
-L PWR_FLAG #FLG01
+L XTAL_DRIVER_TART U2
+U 1 1 5418D7D2
+P 7050 3650
+F 0 "U2" H 7050 3670 50  0000 C CNN
+F 1 "XTAL_DRIVER_TART" H 7050 4030 50  0001 C CNN
+F 2 "MODULE" H 7070 3190 50  0001 C CNN
+F 3 "DOCUMENTATION" H 7050 3270 50  0001 C CNN
+F 4 "XTAL_DRIVER" H 7060 3860 50  0000 C CNN "NAME"
+	1    7050 3650
+	1    0    0    -1
+$EndComp
+$Comp
+L TCXO_TART X1
+U 1 1 5418D7A5
+P 4200 3650
+F 0 "X1" H 4200 3550 50  0000 C CNN
+F 1 "TCXO_TART" H 4210 4190 50  0001 C CNN
+F 2 "MODULE" H 4190 4010 50  0001 C CNN
+F 3 "DOCUMENTATION" H 4200 4100 50  0001 C CNN
+F 4 "TCXO" H 4190 3750 50  0000 C CNN "NAME"
+	1    4200 3650
+	1    0    0    -1
+$EndComp
+$Comp
+L PWR_FLAG #FLG03
 U 1 1 540E3753
 P 8000 3300
-F 0 "#FLG01" H 8000 3395 30  0001 C CNN
+F 0 "#FLG03" H 8000 3395 30  0001 C CNN
 F 1 "PWR_FLAG" H 8000 3480 30  0000 C CNN
 	1    8000 3300
@@
 $EndComp
 $Comp
-L PWR_FLAG #FLG02
+L PWR_FLAG #FLG04
 U 1 1 540E3734
 P 6100 3650
-F 0 "#FLG02" H 6100 3745 30  0001 C CNN
+F 0 "#FLG04" H 6100 3745 30  0001 C CNN
 F 1 "PWR_FLAG" H 6100 3830 30  0000 C CNN
 	1    6100 3650
@@
 	2850 2700 2850 2650
 $Comp
-L VCC #PWR03
+L VCC #PWR05
 U 1 1 5408E937
 P 2850 2650
-F 0 "#PWR03" H 2850 2750 30  0001 C CNN
+F 0 "#PWR05" H 2850 2750 30  0001 C CNN
 F 1 "VCC" H 2850 2750 30  0000 C CNN
 	1    2850 2650
@@
 $EndComp
 $Comp
-L VDD #PWR04
+L VDD #PWR06
 U 1 1 5408E92E
 P 2700 2650
-F 0 "#PWR04" H 2700 2750 30  0001 C CNN
+F 0 "#PWR06" H 2700 2750 30  0001 C CNN
 F 1 "VDD" H 2700 2760 30  0000 C CNN
 	1    2700 2650
@@
 $EndComp
 $Comp
-L VDD #PWR05
+L VDD #PWR07
 U 1 1 5408E909
 P 3250 2650
-F 0 "#PWR05" H 3250 2750 30  0001 C CNN
+F 0 "#PWR07" H 3250 2750 30  0001 C CNN
 F 1 "VDD" H 3250 2760 30  0000 C CNN
 	1    3250 2650
@@
 $EndComp
 $Comp
-L VCC #PWR06
+L VCC #PWR08
 U 1 1 5408E8FA
 P 8000 2650
-F 0 "#PWR06" H 8000 2750 30  0001 C CNN
+F 0 "#PWR08" H 8000 2750 30  0001 C CNN
 F 1 "VCC" H 8000 2750 30  0000 C CNN
 	1    8000 2650
@@
 $EndComp
 $Comp
-L VCC #PWR07
+L VCC #PWR09
 U 1 1 5408E8F1
 P 5850 2650
-F 0 "#PWR07" H 5850 2750 30  0001 C CNN
+F 0 "#PWR09" H 5850 2750 30  0001 C CNN
 F 1 "VCC" H 5850 2750 30  0000 C CNN
 	1    5850 2650
@@
 GND
 $Comp
-L GND #PWR08
+L GND #PWR010
 U 1 1 5408E894
 P 2850 4650
-F 0 "#PWR08" H 2850 4650 30  0001 C CNN
+F 0 "#PWR010" H 2850 4650 30  0001 C CNN
 F 1 "GND" H 2850 4580 30  0001 C CNN
 	1    2850 4650
@@
 $EndComp
 $Comp
-L GND #PWR09
+L GND #PWR011
 U 1 1 5408E850
 P 3250 4650
-F 0 "#PWR09" H 3250 4650 30  0001 C CNN
+F 0 "#PWR011" H 3250 4650 30  0001 C CNN
 F 1 "GND" H 3250 4580 30  0001 C CNN
 	1    3250 4650
@@
 CLK_OUT
 $Comp
-L GND #PWR010
+L GND #PWR012
 U 1 1 5408E752
 P 8000 4600
-F 0 "#PWR010" H 8000 4600 30  0001 C CNN
+F 0 "#PWR012" H 8000 4600 30  0001 C CNN
 F 1 "GND" H 8000 4530 30  0001 C CNN
 	1    8000 4600
@@
 $EndComp
 $Comp
-L GND #PWR011
+L GND #PWR013
 U 1 1 5408E6DB
 P 6100 4600
-F 0 "#PWR011" H 6100 4600 30  0001 C CNN
+F 0 "#PWR013" H 6100 4600 30  0001 C CNN
 F 1 "GND" H 6100 4530 30  0001 C CNN
 	1    6100 4600
@@
 $EndComp
 $Comp
-L GND #PWR012
+L GND #PWR014
 U 1 1 5408E6B1
 P 5850 4600
-F 0 "#PWR012" H 5850 4600 30  0001 C CNN
+F 0 "#PWR014" H 5850 4600 30  0001 C CNN
 F 1 "GND" H 5850 4530 30  0001 C CNN
 	1    5850 4600
@@
 NoConn ~ 6300 3550
 $Comp
-L XTAL_DRIVER U2
-U 1 1 5408E653
-P 7050 3650
-F 0 "U2" H 7050 3550 50  0000 C CNN
-F 1 "XTAL_DRIVER" H 7050 3750 50  0000 C CNN
-F 2 "MODULE" H 7050 3650 50  0001 C CNN
-F 3 "DOCUMENTATION" H 7050 3650 50  0001 C CNN
-	1    7050 3650
-	1    0    0    -1
-$EndComp
-$Comp
-L TCXO X1
-U 1 1 5407E949
-P 4200 3650
-F 0 "X1" H 4200 3550 50  0000 C CNN
-F 1 "TCXO" H 4200 3750 50  0000 C CNN
-F 2 "MODULE" H 4200 3650 50  0001 C CNN
-F 3 "DOCUMENTATION" H 4200 3650 50  0001 C CNN
-	1    4200 3650
-	1    0    0    -1
-$EndComp
-$Comp
-L C C22
+L C C27
 U 1 1 5407E135
 P 8000 4200
-F 0 "C22" H 8050 4300 50  0000 L CNN
+F 0 "C27" H 8050 4300 50  0000 L CNN
 F 1 "0.1u" H 8050 4100 50  0000 L CNN
 	1    8000 4200
@@
 $EndComp
 $Comp
-L R R32
+L R R33
 U 1 1 5407E128
 P 8000 3050
-F 0 "R32" V 8080 3050 50  0000 C CNN
+F 0 "R33" V 8080 3050 50  0000 C CNN
 F 1 "0" V 8000 3050 50  0000 C CNN
 	1    8000 3050
@@
 $EndComp
 $Comp
-L R R31
+L R R32
 U 1 1 5407E121
 P 6100 4200
-F 0 "R31" V 6180 4200 50  0000 C CNN
+F 0 "R32" V 6180 4200 50  0000 C CNN
 F 1 "0" V 6100 4200 50  0000 C CNN
 	1    6100 4200
@@
 $EndComp
 $Comp
-L R R30
+L R R31
 U 1 1 5407E115
 P 5850 4200
-F 0 "R30" V 5930 4200 50  0000 C CNN
+F 0 "R31" V 5930 4200 50  0000 C CNN
 F 1 "10k" V 5850 4200 50  0000 C CNN
 	1    5850 4200
@@
 $EndComp
 $Comp
-L R R29
+L R R30
 U 1 1 5407E105
 P 5850 3050
-F 0 "R29" V 5930 3050 50  0000 C CNN
+F 0 "R30" V 5930 3050 50  0000 C CNN
 F 1 "10k" V 5850 3050 50  0000 C CNN
 	1    5850 3050
@@
 $EndComp
 $Comp
-L C C21
+L C C26
 U 1 1 5407E0F8
 P 5450 3750
-F 0 "C21" H 5500 3850 50  0000 L CNN
+F 0 "C26" H 5500 3850 50  0000 L CNN
 F 1 "2200p" H 5500 3650 50  0000 L CNN
 	1    5450 3750

Commit message: Work progresses on new base station board
Connections:
- net CLK_FPGA: now also U2.6 (Y); no longer U2.4 (X2)
- net CLK_OUT: now also U2.4 (X2); no longer U2.6 (Y)
Changed lines of the file:
@@
-EESchema Schematic File Version 2  date Wed 17 Sep 2014 15:47:12 NZST
+EESchema Schematic File Version 2  date Tue 23 Sep 2014 15:10:21 NZST
 LIBS:power
 LIBS:device
@@
 LIBS:valves
 LIBS:TART
+LIBS:IC_raspberry
 LIBS:base_station_integrated-cache
 EELAYER 25  0
@@
 Sheet 7 7
 Title ""
-Date "17 sep 2014"
+Date "23 sep 2014"
 Rev ""
 Comp ""
@@
 	1    0    0    -1
 $EndComp
+Text HLabel 8300 3550 2    60   Input ~ 0
+CLK_FPGA
 Text HLabel 8300 3750 2    60   Input ~ 0
-CLK_FPGA
-Text HLabel 8300 3550 2    60   Input ~ 0
 CLK_OUT
 $Comp

Commit message: Routine backup
Parts:
- renumbered C26 to C32, C27 to C33
Changed lines of the file:
@@
-EESchema Schematic File Version 2  date Tue 23 Sep 2014 15:10:21 NZST
+EESchema Schematic File Version 2  date Wed 24 Sep 2014 17:40:46 NZST
 LIBS:power
 LIBS:device
@@
 Sheet 7 7
 Title ""
-Date "23 sep 2014"
+Date "24 sep 2014"
 Rev ""
 Comp ""
@@
 $EndComp
 $Comp
-L PWR_FLAG #FLG03
+L PWR_FLAG #FLG04
 U 1 1 540E3753
 P 8000 3300
-F 0 "#FLG03" H 8000 3395 30  0001 C CNN
+F 0 "#FLG04" H 8000 3395 30  0001 C CNN
 F 1 "PWR_FLAG" H 8000 3480 30  0000 C CNN
 	1    8000 3300
@@
 $EndComp
 $Comp
-L PWR_FLAG #FLG04
+L PWR_FLAG #FLG05
 U 1 1 540E3734
 P 6100 3650
-F 0 "#FLG04" H 6100 3745 30  0001 C CNN
+F 0 "#FLG05" H 6100 3745 30  0001 C CNN
 F 1 "PWR_FLAG" H 6100 3830 30  0000 C CNN
 	1    6100 3650
@@
 	2850 2700 2850 2650
 $Comp
-L VCC #PWR05
+L VCC #PWR06
 U 1 1 5408E937
 P 2850 2650
-F 0 "#PWR05" H 2850 2750 30  0001 C CNN
+F 0 "#PWR06" H 2850 2750 30  0001 C CNN
 F 1 "VCC" H 2850 2750 30  0000 C CNN
 	1    2850 2650
@@
 $EndComp
 $Comp
-L VDD #PWR06
+L VDD #PWR07
 U 1 1 5408E92E
 P 2700 2650
-F 0 "#PWR06" H 2700 2750 30  0001 C CNN
+F 0 "#PWR07" H 2700 2750 30  0001 C CNN
 F 1 "VDD" H 2700 2760 30  0000 C CNN
 	1    2700 2650
@@
 $EndComp
 $Comp
-L VDD #PWR07
+L VDD #PWR08
 U 1 1 5408E909
 P 3250 2650
-F 0 "#PWR07" H 3250 2750 30  0001 C CNN
+F 0 "#PWR08" H 3250 2750 30  0001 C CNN
 F 1 "VDD" H 3250 2760 30  0000 C CNN
 	1    3250 2650
@@
 $EndComp
 $Comp
-L VCC #PWR08
+L VCC #PWR09
 U 1 1 5408E8FA
 P 8000 2650
-F 0 "#PWR08" H 8000 2750 30  0001 C CNN
+F 0 "#PWR09" H 8000 2750 30  0001 C CNN
 F 1 "VCC" H 8000 2750 30  0000 C CNN
 	1    8000 2650
@@
 $EndComp
 $Comp
-L VCC #PWR09
+L VCC #PWR010
 U 1 1 5408E8F1
 P 5850 2650
-F 0 "#PWR09" H 5850 2750 30  0001 C CNN
+F 0 "#PWR010" H 5850 2750 30  0001 C CNN
 F 1 "VCC" H 5850 2750 30  0000 C CNN
 	1    5850 2650
@@
 GND
 $Comp
-L GND #PWR010
+L GND #PWR011
 U 1 1 5408E894
 P 2850 4650
-F 0 "#PWR010" H 2850 4650 30  0001 C CNN
+F 0 "#PWR011" H 2850 4650 30  0001 C CNN
 F 1 "GND" H 2850 4580 30  0001 C CNN
 	1    2850 4650
@@
 $EndComp
 $Comp
-L GND #PWR011
+L GND #PWR012
 U 1 1 5408E850
 P 3250 4650
-F 0 "#PWR011" H 3250 4650 30  0001 C CNN
+F 0 "#PWR012" H 3250 4650 30  0001 C CNN
 F 1 "GND" H 3250 4580 30  0001 C CNN
 	1    3250 4650
@@
 CLK_OUT
 $Comp
-L GND #PWR012
+L GND #PWR013
 U 1 1 5408E752
 P 8000 4600
-F 0 "#PWR012" H 8000 4600 30  0001 C CNN
+F 0 "#PWR013" H 8000 4600 30  0001 C CNN
 F 1 "GND" H 8000 4530 30  0001 C CNN
 	1    8000 4600
@@
 $EndComp
 $Comp
-L GND #PWR013
+L GND #PWR014
 U 1 1 5408E6DB
 P 6100 4600
-F 0 "#PWR013" H 6100 4600 30  0001 C CNN
+F 0 "#PWR014" H 6100 4600 30  0001 C CNN
 F 1 "GND" H 6100 4530 30  0001 C CNN
 	1    6100 4600
@@
 $EndComp
 $Comp
-L GND #PWR014
+L GND #PWR015
 U 1 1 5408E6B1
 P 5850 4600
-F 0 "#PWR014" H 5850 4600 30  0001 C CNN
+F 0 "#PWR015" H 5850 4600 30  0001 C CNN
 F 1 "GND" H 5850 4530 30  0001 C CNN
 	1    5850 4600
@@
 NoConn ~ 6300 3550
 $Comp
-L C C27
+L C C33
 U 1 1 5407E135
 P 8000 4200
-F 0 "C27" H 8050 4300 50  0000 L CNN
+F 0 "C33" H 8050 4300 50  0000 L CNN
 F 1 "0.1u" H 8050 4100 50  0000 L CNN
 	1    8000 4200
@@
 $EndComp
 $Comp
-L C C26
+L C C32
 U 1 1 5407E0F8
 P 5450 3750
-F 0 "C26" H 5500 3850 50  0000 L CNN
+F 0 "C32" H 5500 3850 50  0000 L CNN
 F 1 "2200p" H 5500 3650 50  0000 L CNN
 	1    5450 3750
