File: hardware/pcb/kicad/base_station_clock.sch (KiCad schematic (older format))
At the start: 8 parts, among them U2 XTAL_DRIVER_TART, X1 TCXO_TART

Commit message: Made component references more logical - very similar to eagle version
Parts:
- renumbered C33 to C25, C32 to C26, U2 to IC26, R33 to R29, R32 to R30, R30 to R32
Changed lines of the file:
@@
 Sheet 7 7
 Title ""
-Date "4 dec 2014"
+Date "8 dec 2014"
 Rev ""
 Comp ""
@@
 $EndDescr
 $Comp
-L XTAL_DRIVER_TART U2
+L XTAL_DRIVER_TART IC26
 U 1 1 5418D7D2
 P 7050 3650
-F 0 "U2" H 7050 3670 50  0000 C CNN
+F 0 "IC26" H 7050 3670 50  0000 C CNN
 F 1 "XTAL_DRIVER_TART" H 7050 4030 50  0001 C CNN
 F 2 "MODULE" H 7070 3190 50  0001 C CNN
@@
 NoConn ~ 6300 3550
 $Comp
-L C C33
+L C C25
 U 1 1 5407E135
 P 8000 4200
-F 0 "C33" H 8050 4300 50  0000 L CNN
+F 0 "C25" H 8050 4300 50  0000 L CNN
 F 1 "0.1u" H 8050 4100 50  0000 L CNN
 F 2 "" H 8000 4200 60  0001 C CNN
@@
 $EndComp
 $Comp
-L R R33
+L R R29
 U 1 1 5407E128
 P 8000 3050
-F 0 "R33" V 8080 3050 50  0000 C CNN
+F 0 "R29" V 8080 3050 50  0000 C CNN
 F 1 "0" V 8000 3050 50  0000 C CNN
 F 2 "" H 8000 3050 60  0001 C CNN
@@
 $EndComp
 $Comp
-L R R32
+L R R30
 U 1 1 5407E121
 P 6100 4200
-F 0 "R32" V 6180 4200 50  0000 C CNN
+F 0 "R30" V 6180 4200 50  0000 C CNN
 F 1 "0" V 6100 4200 50  0000 C CNN
 F 2 "" H 6100 4200 60  0001 C CNN
@@
 $EndComp
 $Comp
-L R R30
+L R R32
 U 1 1 5407E105
 P 5850 3050
-F 0 "R30" V 5930 3050 50  0000 C CNN
+F 0 "R32" V 5930 3050 50  0000 C CNN
 F 1 "10k" V 5850 3050 50  0000 C CNN
 F 2 "" H 5850 3050 60  0001 C CNN
@@
 $EndComp
 $Comp
-L C C32
+L C C26
 U 1 1 5407E0F8
 P 5450 3750
-F 0 "C32" H 5500 3850 50  0000 L CNN
+F 0 "C26" H 5500 3850 50  0000 L CNN
 F 1 "2200p" H 5500 3650 50  0000 L CNN
 F 2 "" H 5450 3750 60  0001 C CNN
