File: hardware/pcb/kicad/base_station_integrated.sch (KiCad schematic (older format))
At the start: 5 parts, among them U1 MEGAWING_HALF_P1_MEGAWING_HAL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

Commit message: Getting libraries to work...
Parts:
- removed JP1, JP2, JP3, JP4: JUMPER3, symbol JUMPER3
- removed U1: MEGAWING_HALF_P1_MEGAWING_HALF_NOHOLES_P1, symbol MEGAWING_HALF_P1_MEGAWING_HALF_NOHOLES_P1
- added JP1, JP2, JP3, JP4: JUMP_OR_TART, symbol JUMP_OR_TART
- added U1: PAPILIO_TART, symbol PAPILIO_TART
Connections:
- wire segments 98 -> 99

Commit message: Work progresses on new base station board
Parts:
- removed JP1, JP2, JP3, JP4: JUMP_OR_TART, symbol JUMP_OR_TART
- added P1: CONN_20X2, symbol CONN_20X2
Connections:
- net +5V: now also P1.2 (P2), P1.4 (P4)
- net GND: now also P1.14 (P14), P1.20 (P20), P1.6 (P6), P1.9 (P9)
- net MOSI: now reaches U1.A10
- net MOSI: now also P1.19 (P19)
- net SCLK: now reaches U1.A12
- net SCLK: now also P1.23 (P23)
- net MISO: now reaches U1.B6
- net MISO: now also P1.21 (P21)
- no-connect marks 13 -> 47

Commit message: Routine backup
Connections:
- net +5V: no longer P1.2 (P2), P1.4 (P4)
- new net +5V_PI: P1.2 (P2), P1.4 (P4)
Other:
- moved on the sheet: P1
