File: hardware/pcb/kicad/base_station_power_supply.sch (KiCad schematic (older format))
At the start: 14 parts, among them U3 POWER_JACKPTH_POWER_JACK_PTH

Commit message: Getting libraries to work...
Parts:
- removed D1: SHOTTKY-BIDR, symbol SHOTTKY-BIDR
- removed D2: BRIDGE, symbol BRIDGE
- removed D3: DIODESCH, symbol DIODESCH
- removed REG1: OKI-78SR-5/1.5, symbol OKI-78SR-5/1.5
- removed REG2: SPX3940, symbol SPX3940
- removed U3: POWER_JACKPTH_POWER_JACK_PTH, symbol POWER_JACKPTH_POWER_JACK_PTH
- added CON1: POWER_JACK_TART, symbol POWER_JACK_TART
- added D1: TVS_DIODE_BI_TART, symbol TVS_DIODE_BI_TART
- added D2: TVS_DIODE_UNI_TART, symbol TVS_DIODE_UNI_TART
- added IC1: BRIDGE_TART, symbol BRIDGE_TART
- added REG1: OK1-78SR_TART, symbol OK1-78SR_TART
- added REG2: SPX3940_TART, symbol SPX3940_TART
- C1: renamed from C23; footprint (none) -> E5-10,5_TART
- C3: renamed from C25; footprint (none) -> E5-10,5_TART
- C5: renamed from C27; footprint (none) -> E2-5_TART
- renumbered C24 to C2, C26 to C4, D4 to D3, R33 to R1
Connections:
- net labels added: +5V
- wire segments 33 -> 32
Changed lines of the file:
@@
-EESchema Schematic File Version 2  date Tue 09 Sep 2014 11:32:54 NZST
+EESchema Schematic File Version 2  date Wed 17 Sep 2014 15:47:12 NZST
 LIBS:power
 LIBS:device
@@
 LIBS:valves
 LIBS:TART
-LIBS:Papilio
 LIBS:base_station_integrated-cache
 EELAYER 25  0
@@
 $Descr A4 11700 8267
 encoding utf-8
-Sheet 7 7
+Sheet 2 7
 Title ""
-Date "8 sep 2014"
+Date "17 sep 2014"
 Rev ""
 Comp ""
@@
 $EndDescr
 $Comp
-L PWR_FLAG #FLG013
+L SPX3940_TART REG2
+U 1 1 5419032C
+P 8450 3650
+F 0 "REG2" H 8600 3434 60  0000 C CNN
+F 1 "SPX3940_TART" H 8450 3960 60  0001 C CNN
+F 4 "SPX3940" H 8450 3854 60  0000 C CNN "NAME"
+	1    8450 3650
+	1    0    0    -1
+$EndComp
+$Comp
+L OK1-78SR_TART REG1
+U 1 1 54190317
+P 6950 3650
+F 0 "REG1" H 7100 3434 60  0000 C CNN
+F 1 "OK1-78SR_TART" H 6950 3960 60  0001 C CNN
+F 4 "OKI-78SR" H 6950 3854 60  0000 C CNN "NAME"
+	1    6950 3650
+	1    0    0    -1
+$EndComp
+$Comp
+L POWER_JACK_TART CON1
+U 1 1 5418E80C
+P 1600 3700
+F 0 "CON1" H 1850 4000 60  0000 C CNN
+F 1 "POWER_JACK_TART" H 1600 4110 60  0001 C CNN
+F 4 "POWER_JACK" H 1720 3600 60  0000 C CNN "NAME"
+	1    1600 3700
+	1    0    0    -1
+$EndComp
+$Comp
+L TVS_DIODE_BI_TART D1
+U 1 1 5418D706
+P 2550 3600
+F 0 "D1" H 2550 3725 40  0000 C CNN
+F 1 "TVS_DIODE_BI_TART" H 2530 3795 40  0001 C CNN
+F 4 "TVS_DIODE_BI" H 2560 3465 40  0000 C CNN "NAME"
+	1    2550 3600
+	0    -1   -1   0
+$EndComp
+$Comp
+L TVS_DIODE_UNI_TART D2
+U 1 1 5418D6C0
+P 5600 4150
+F 0 "D2" H 5600 4250 40  0000 C CNN
+F 1 "TVS_DIODE_UNI_TART" H 5590 4310 40  0001 C CNN
+F 4 "TVS_DIODE_UNI" H 5600 4040 40  0000 C CNN "NAME"
+	1    5600 4150
+	0    -1   -1   0
+$EndComp
+$Comp
+L BRIDGE_TART IC1
+U 1 1 5418D689
+P 4000 3600
+F 0 "IC1" H 4000 3650 70  0000 C CNN
+F 1 "BRIDGE_TART" H 4550 4550 60  0001 C CNN
+F 4 "MICRO COMMERCIAL" H 4700 4450 60  0001 C CNN "MANUFAC"
+F 5 "MB16S-TP" H 4500 4350 60  0001 C CNN "MAN_PART"
+F 6 "MB16S-TPMSCT-ND" H 4700 4250 60  0001 C CNN "DIGIKEY"
+F 7 "BRIDGE" H 4000 3550 70  0000 C CNN "NAME"
+	1    4000 3600
+	1    0    0    -1
+$EndComp
+Wire Wire Line
+	7450 2350 7450 3900
+Wire Wire Line
+	6350 3350 6350 3600
+Wire Wire Line
+	9800 4600 3150 4600
+Wire Wire Line
+	4850 3600 5850 3600
+Connection ~ 5600 4600
+Wire Wire Line
+	5600 4300 5600 4850
+Connection ~ 4950 3600
+Wire Wire Line
+	4950 3900 4950 3600
+Connection ~ 5300 4600
+Wire Wire Line
+	5300 4600 5300 4300
+Wire Wire Line
+	3150 4600 3150 3600
+Connection ~ 2550 2750
+Wire Wire Line
+	4000 2750 2200 2750
+Wire Wire Line
+	2200 2750 2200 3500
+Wire Wire Line
+	2550 3350 2550 2750
+Wire Wire Line
+	2200 3500 2000 3500
+Wire Wire Line
+	6350 3600 6550 3600
+Wire Wire Line
+	9800 3900 9800 3600
+Wire Wire Line
+	9800 3600 9700 3600
+Connection ~ 7900 4600
+Wire Wire Line
+	7900 4600 7900 4300
+Connection ~ 6950 4600
+Wire Wire Line
+	8950 4600 8950 4300
+Wire Wire Line
+	6950 4600 6950 3900
+Connection ~ 7450 3600
+Wire Wire Line
+	7350 3600 8050 3600
+Wire Wire Line
+	7900 3600 7900 3900
+Connection ~ 7900 3600
+Wire Wire Line
+	7450 4600 7450 4300
+Connection ~ 7450 4600
+Wire Wire Line
+	9200 3600 8850 3600
+Connection ~ 8950 3600
+Connection ~ 8950 4600
+Wire Wire Line
+	2000 3700 2200 3700
+Wire Wire Line
+	2550 3850 2550 4450
+Wire Wire Line
+	2200 3700 2200 4450
+Wire Wire Line
+	2200 4450 4000 4450
+Connection ~ 2550 4450
+Wire Wire Line
+	4950 4300 4950 4600
+Connection ~ 4950 4600
+Wire Wire Line
+	5300 3600 5300 3900
+Connection ~ 5300 3600
+Wire Wire Line
+	5600 3900 5600 2350
+Connection ~ 5600 3600
+Wire Wire Line
+	8950 3900 8950 2350
+Wire Wire Line
+	8450 4600 8450 3900
+Connection ~ 8450 4600
+Wire Wire Line
+	9800 4850 9800 4300
+Connection ~ 9800 4600
+Text HLabel 7450 2350 1    60   Input ~ 0
++5V
+$Comp
+L PWR_FLAG #FLG01
 U 1 1 540E3627
 P 9800 4850
-F 0 "#FLG013" H 9800 4945 30  0001 C CNN
+F 0 "#FLG01" H 9800 4945 30  0001 C CNN
 F 1 "PWR_FLAG" H 9800 5030 30  0000 C CNN
 	1    9800 4850
 	-1   0    0    1
 $EndComp
-Connection ~ 9800 4600
-Wire Wire Line
-	9800 4850 9800 4300
-Connection ~ 8450 4600
-Wire Wire Line
-	8450 4600 8450 3900
-Wire Wire Line
-	8950 3900 8950 2350
-Connection ~ 5600 3600
-Wire Wire Line
-	5600 3900 5600 2350
-Wire Wire Line
-	5650 4100 5600 4100
-Connection ~ 5300 3600
-Wire Wire Line
-	5300 3600 5300 3900
-Connection ~ 4950 4600
-Wire Wire Line
-	4950 4300 4950 4600
-Connection ~ 2550 4450
-Wire Wire Line
-	4000 4450 2200 4450
-Wire Wire Line
-	2200 4450 2200 3700
-Wire Wire Line
-	2550 3850 2550 4450
-Wire Wire Line
-	2200 3700 2000 3700
-Connection ~ 8950 4600
-Connection ~ 8950 3600
-Wire Wire Line
-	9200 3600 8850 3600
-Connection ~ 7450 4600
-Wire Wire Line
-	7450 4600 7450 4300
-Connection ~ 7900 3600
-Wire Wire Line
-	7900 3600 7900 3900
-Wire Wire Line
-	7350 3600 8050 3600
-Wire Wire Line
-	7450 3900 7450 3600
-Connection ~ 7450 3600
-Wire Wire Line
-	6950 4600 6950 3900
-Wire Wire Line
-	8950 4600 8950 4300
-Connection ~ 6950 4600
-Wire Wire Line
-	7900 4600 7900 4300
-Connection ~ 7900 4600
-Wire Wire Line
-	9700 3600 9800 3600
-Wire Wire Line
-	9800 3600 9800 3900
-Wire Wire Line
-	6550 3600 6350 3600
-Wire Wire Line
-	2000 3500 2200 3500
-Wire Wire Line
-	2550 3350 2550 2750
-Wire Wire Line
-	2200 3500 2200 2750
-Wire Wire Line
-	2200 2750 4000 2750
-Connection ~ 2550 2750
-Wire Wire Line
-	3150 3600 3150 4600
-Wire Wire Line
-	5300 4600 5300 4300
-Connection ~ 5300 4600
-Wire Wire Line
-	4950 3900 4950 3600
-Connection ~ 4950 3600
-Wire Wire Line
-	5600 4300 5600 4850
-Connection ~ 5600 4600
-Wire Wire Line
-	4850 3600 5850 3600
-Wire Wire Line
-	3150 4600 9800 4600
-Wire Wire Line
-	6350 3600 6350 3350
-$Comp
-L PWR_FLAG #FLG014
+$Comp
+L PWR_FLAG #FLG02
 U 1 1 540E3477
 P 6350 3350
-F 0 "#FLG014" H 6350 3445 30  0001 C CNN
+F 0 "#FLG02" H 6350 3445 30  0001 C CNN
 F 1 "PWR_FLAG" H 6350 3530 30  0000 C CNN
 	1    6350 3350
@@
 +24V
 $Comp
-L DIODESCH D3
-U 1 1 5407CBCB
-P 5600 4100
-F 0 "D3" H 5600 4200 40  0000 C CNN
-F 1 "DIODESCH" H 5600 4000 40  0000 C CNN
-	1    5600 4100
-	0    -1   -1   0
-$EndComp
-$Comp
-L C C24
+L C C2
 U 1 1 5407CB7A
 P 5300 4100
-F 0 "C24" H 5350 4200 50  0000 L CNN
+F 0 "C2" H 5350 4200 50  0000 L CNN
 F 1 "0.1u" H 5350 4000 50  0000 L CNN
 	1    5300 4100
@@
 $EndComp
 $Comp
-L CP1 C23
+L CP1 C1
 U 1 1 5407CB6C
 P 4950 4100
-F 0 "C23" H 5000 4200 50  0000 L CNN
+F 0 "C1" H 5000 4200 50  0000 L CNN
 F 1 "100u" H 5000 4000 50  0000 L CNN
+F 2 "E5-10,5_TART" H 4950 4100 60  0001 C CNN
 	1    4950 4100
-	1    0    0    -1
-$EndComp
-$Comp
-L BRIDGE D2
-U 1 1 5407CAA3
-P 4000 3600
-F 0 "D2" H 4000 3650 70  0000 C CNN
-F 1 "BRIDGE" H 4000 3550 70  0000 C CNN
-	1    4000 3600
-	1    0    0    -1
-$EndComp
-$Comp
-L SHOTTKY-BIDR D1
-U 1 1 5407CA3E
-P 2550 3600
-F 0 "D1" H 2500 3725 40  0000 C CNN
-F 1 "SHOTTKY-BIDR" H 2550 3475 40  0000 C CNN
-	1    2550 3600
-	0    -1   -1   0
-$EndComp
-$Comp
-L POWER_JACKPTH_POWER_JACK_PTH U3
-U 1 1 5407A835
-P 1600 3700
-F 0 "U3" H 1600 3700 60  0001 C CNN
-F 1 "POWER_JACKPTH_POWER_JACK_PTH" H 1600 3700 60  0001 C CNN
-	1    1600 3700
 	1    0    0    -1
 $EndComp
@@
 $EndComp
 $Comp
-L LED D4
+L LED D3
 U 1 1 5407A3D9
 P 9800 4100
-F 0 "D4" H 9800 4200 50  0000 C CNN
+F 0 "D3" H 9800 4200 50  0000 C CNN
 F 1 "LED" H 9800 4000 50  0000 C CNN
 	1    9800 4100
@@
 $EndComp
 $Comp
-L R R33
+L R R1
 U 1 1 5407A3AD
 P 9450 3600
-F 0 "R33" V 9530 3600 50  0000 C CNN
+F 0 "R1" V 9530 3600 50  0000 C CNN
 F 1 "R" V 9450 3600 50  0000 C CNN
 	1    9450 3600
@@
 $EndComp
 $Comp
-L CP1 C27
+L CP1 C5
 U 1 1 5407A35C
 P 8950 4100
-F 0 "C27" H 9000 4200 50  0000 L CNN
+F 0 "C5" H 9000 4200 50  0000 L CNN
 F 1 "10u" H 9000 4000 50  0000 L CNN
+F 2 "E2-5_TART" H 8950 4100 60  0001 C CNN
 	1    8950 4100
 	1    0    0    -1
 $EndComp
 $Comp
-L C C26
+L C C4
 U 1 1 5407A2F7
 P 7900 4100
-F 0 "C26" H 7950 4200 50  0000 L CNN
+F 0 "C4" H 7950 4200 50  0000 L CNN
 F 1 "0.1u" H 7950 4000 50  0000 L CNN
 	1    7900 4100
@@
 $EndComp
 $Comp
-L CP1 C25
+L CP1 C3
 U 1 1 5407A2C8
 P 7450 4100
-F 0 "C25" H 7500 4200 50  0000 L CNN
+F 0 "C3" H 7500 4200 50  0000 L CNN
 F 1 "10u" H 7500 4000 50  0000 L CNN
+F 2 "E5-10,5_TART" H 7450 4100 60  0001 C CNN
 	1    7450 4100
 	1    0    0    -1
 $EndComp
-$Comp
-L SPX3940 REG2
-U 1 1 5407A27B
-P 8450 3650
-F 0 "REG2" H 8600 3454 60  0000 C CNN
-F 1 "SPX3940" H 8450 3850 60  0000 C CNN
-	1    8450 3650
-	1    0    0    -1
-$EndComp
-$Comp
-L OKI-78SR-5/1.5 REG1
-U 1 1 5407A0C8
-P 6950 3650
-F 0 "REG1" H 7100 3454 60  0000 C CNN
-F 1 "OKI-78SR-5/1.5" H 6950 3850 60  0000 C CNN
-	1    6950 3650
-	1    0    0    -1
-$EndComp

Commit message: Routine backup
Parts:
- added C1: 10u, E5-10,5_TART, symbol CP1
- added C2: 0.1u, symbol C
- added F1: FUSE, symbol FUSE
- added REG1: OK1-78SR_TART, symbol OK1-78SR_TART
- renumbered C1 to C3, C2 to C4, C3 to C5, C4 to C6, C5 to C7, F1 to F2, REG1 to REG2, REG2 to REG3
Connections:
- net labels added: +5V_PI
- wire segments 32 -> 45
Changed lines of the file:
@@
-EESchema Schematic File Version 2  date Tue 23 Sep 2014 15:10:21 NZST
+EESchema Schematic File Version 2  date Wed 24 Sep 2014 17:40:46 NZST
 LIBS:power
 LIBS:device
@@
 Sheet 2 7
 Title ""
-Date "23 sep 2014"
+Date "24 sep 2014"
 Rev ""
 Comp ""
@@
 $EndDescr
 $Comp
-L SPX3940_TART REG2
+L FUSE F1
+U 1 1 5421F748
+P 2350 5750
+F 0 "F1" H 2450 5800 40  0000 C CNN
+F 1 "FUSE" H 2250 5700 40  0000 C CNN
+	1    2350 5750
+	1    0    0    -1
+$EndComp
+Wire Wire Line
+	5600 2350 5600 3950
+Wire Wire Line
+	4650 6550 4650 6400
+Connection ~ 3700 6400
+Wire Wire Line
+	3200 6050 3200 6400
+Wire Wire Line
+	2100 5750 1850 5750
+Wire Wire Line
+	3700 5850 3700 5750
+Wire Wire Line
+	3700 6250 3700 6400
+Connection ~ 4150 5750
+Wire Wire Line
+	4150 5750 4150 5850
+Connection ~ 3700 5750
+Wire Wire Line
+	4150 6400 4150 6250
+Connection ~ 4150 6400
+Wire Wire Line
+	2800 5750 2600 5750
+Wire Wire Line
+	2600 5750 2600 5500
+Wire Wire Line
+	7450 3900 7450 2350
+Wire Wire Line
+	6350 3350 6350 3600
+Wire Wire Line
+	9800 4600 3150 4600
+Wire Wire Line
+	5850 3600 4850 3600
+Connection ~ 5600 4600
+Connection ~ 4950 3600
+Wire Wire Line
+	4950 3600 4950 3900
+Connection ~ 5300 4600
+Wire Wire Line
+	5300 4600 5300 4300
+Wire Wire Line
+	3150 4600 3150 3600
+Connection ~ 2550 2750
+Wire Wire Line
+	4000 2750 2200 2750
+Wire Wire Line
+	2200 2750 2200 3500
+Wire Wire Line
+	2550 3350 2550 2750
+Wire Wire Line
+	2200 3500 2000 3500
+Wire Wire Line
+	6350 3600 6550 3600
+Wire Wire Line
+	9800 3900 9800 3600
+Wire Wire Line
+	9800 3600 9700 3600
+Connection ~ 7900 4600
+Wire Wire Line
+	7900 4600 7900 4300
+Connection ~ 6950 4600
+Wire Wire Line
+	8950 4600 8950 4300
+Wire Wire Line
+	6950 4600 6950 3900
+Connection ~ 7450 3600
+Wire Wire Line
+	8050 3600 7350 3600
+Wire Wire Line
+	7900 3900 7900 3600
+Connection ~ 7900 3600
+Wire Wire Line
+	7450 4600 7450 4300
+Connection ~ 7450 4600
+Wire Wire Line
+	8850 3600 9200 3600
+Connection ~ 8950 3600
+Connection ~ 8950 4600
+Wire Wire Line
+	2000 3700 2200 3700
+Wire Wire Line
+	2550 3850 2550 4450
+Wire Wire Line
+	2200 3700 2200 4450
+Wire Wire Line
+	2200 4450 4000 4450
+Connection ~ 2550 4450
+Wire Wire Line
+	4950 4300 4950 4600
+Connection ~ 4950 4600
+Wire Wire Line
+	5300 3600 5300 3900
+Connection ~ 5300 3600
+Connection ~ 5600 3600
+Wire Wire Line
+	8950 2350 8950 3900
+Wire Wire Line
+	8450 4600 8450 3900
+Connection ~ 8450 4600
+Wire Wire Line
+	9800 4300 9800 4850
+Connection ~ 9800 4600
+Wire Wire Line
+	1850 5750 1850 5100
+Wire Wire Line
+	4650 5600 4650 5750
+Wire Wire Line
+	4650 5750 3600 5750
+Wire Wire Line
+	3200 6400 4650 6400
+Wire Wire Line
+	5600 4350 5600 4600
+Text HLabel 4650 6550 3    60   Input ~ 0
+GND
+Text HLabel 4650 5600 1    60   Input ~ 0
++5V_PI
+$Comp
+L CP1 C1
+U 1 1 5421F74A
+P 3700 6050
+F 0 "C1" H 3750 6150 50  0000 L CNN
+F 1 "10u" H 3750 5950 50  0000 L CNN
+F 2 "E5-10,5_TART" H 3700 6050 60  0001 C CNN
+	1    3700 6050
+	1    0    0    -1
+$EndComp
+$Comp
+L C C2
+U 1 1 5421F749
+P 4150 6050
+F 0 "C2" H 4200 6150 50  0000 L CNN
+F 1 "0.1u" H 4200 5950 50  0000 L CNN
+	1    4150 6050
+	1    0    0    -1
+$EndComp
+Text HLabel 1850 5100 1    60   Input ~ 0
++24V
+$Comp
+L PWR_FLAG #FLG01
+U 1 1 5421F747
+P 2600 5500
+F 0 "#FLG01" H 2600 5595 30  0001 C CNN
+F 1 "PWR_FLAG" H 2600 5680 30  0000 C CNN
+	1    2600 5500
+	1    0    0    -1
+$EndComp
+$Comp
+L OK1-78SR_TART REG1
+U 1 1 5421F746
+P 3200 5800
+F 0 "REG1" H 3350 5584 60  0000 C CNN
+F 1 "OK1-78SR_TART" H 3200 6110 60  0001 C CNN
+F 4 "OKI-78SR" H 3200 6004 60  0000 C CNN "NAME"
+	1    3200 5800
+	1    0    0    -1
+$EndComp
+$Comp
+L SPX3940_TART REG3
 U 1 1 5419032C
 P 8450 3650
-F 0 "REG2" H 8600 3434 60  0000 C CNN
+F 0 "REG3" H 8600 3434 60  0000 C CNN
 F 1 "SPX3940_TART" H 8450 3960 60  0001 C CNN
 F 4 "SPX3940" H 8450 3854 60  0000 C CNN "NAME"
@@
 $EndComp
 $Comp
-L OK1-78SR_TART REG1
+L OK1-78SR_TART REG2
 U 1 1 54190317
 P 6950 3650
-F 0 "REG1" H 7100 3434 60  0000 C CNN
+F 0 "REG2" H 7100 3434 60  0000 C CNN
 F 1 "OK1-78SR_TART" H 6950 3960 60  0001 C CNN
 F 4 "OKI-78SR" H 6950 3854 60  0000 C CNN "NAME"
@@
 	1    0    0    -1
 $EndComp
-Wire Wire Line
-	7450 2350 7450 3900
-Wire Wire Line
-	6350 3350 6350 3600
-Wire Wire Line
-	9800 4600 3150 4600
-Wire Wire Line
-	4850 3600 5850 3600
-Connection ~ 5600 4600
-Wire Wire Line
-	5600 4300 5600 4850
-Connection ~ 4950 3600
-Wire Wire Line
-	4950 3900 4950 3600
-Connection ~ 5300 4600
-Wire Wire Line
-	5300 4600 5300 4300
-Wire Wire Line
-	3150 4600 3150 3600
-Connection ~ 2550 2750
-Wire Wire Line
-	4000 2750 2200 2750
-Wire Wire Line
-	2200 2750 2200 3500
-Wire Wire Line
-	2550 3350 2550 2750
-Wire Wire Line
-	2200 3500 2000 3500
-Wire Wire Line
-	6350 3600 6550 3600
-Wire Wire Line
-	9800 3900 9800 3600
-Wire Wire Line
-	9800 3600 9700 3600
-Connection ~ 7900 4600
-Wire Wire Line
-	7900 4600 7900 4300
-Connection ~ 6950 4600
-Wire Wire Line
-	8950 4600 8950 4300
-Wire Wire Line
-	6950 4600 6950 3900
-Connection ~ 7450 3600
-Wire Wire Line
-	7350 3600 8050 3600
-Wire Wire Line
-	7900 3600 7900 3900
-Connection ~ 7900 3600
-Wire Wire Line
-	7450 4600 7450 4300
-Connection ~ 7450 4600
-Wire Wire Line
-	9200 3600 8850 3600
-Connection ~ 8950 3600
-Connection ~ 8950 4600
-Wire Wire Line
-	2000 3700 2200 3700
-Wire Wire Line
-	2550 3850 2550 4450
-Wire Wire Line
-	2200 3700 2200 4450
-Wire Wire Line
-	2200 4450 4000 4450
-Connection ~ 2550 4450
-Wire Wire Line
-	4950 4300 4950 4600
-Connection ~ 4950 4600
-Wire Wire Line
-	5300 3600 5300 3900
-Connection ~ 5300 3600
-Wire Wire Line
-	5600 3900 5600 2350
-Connection ~ 5600 3600
-Wire Wire Line
-	8950 3900 8950 2350
-Wire Wire Line
-	8450 4600 8450 3900
-Connection ~ 8450 4600
-Wire Wire Line
-	9800 4850 9800 4300
-Connection ~ 9800 4600
 Text HLabel 7450 2350 1    60   Input ~ 0
 +5V
 $Comp
-L PWR_FLAG #FLG01
+L PWR_FLAG #FLG02
 U 1 1 540E3627
 P 9800 4850
-F 0 "#FLG01" H 9800 4945 30  0001 C CNN
+F 0 "#FLG02" H 9800 4945 30  0001 C CNN
 F 1 "PWR_FLAG" H 9800 5030 30  0000 C CNN
 	1    9800 4850
@@
 $EndComp
 $Comp
-L PWR_FLAG #FLG02
+L PWR_FLAG #FLG03
 U 1 1 540E3477
 P 6350 3350
-F 0 "#FLG02" H 6350 3445 30  0001 C CNN
+F 0 "#FLG03" H 6350 3445 30  0001 C CNN
 F 1 "PWR_FLAG" H 6350 3530 30  0000 C CNN
 	1    6350 3350
@@
 +24V
 $Comp
-L C C2
+L C C4
 U 1 1 5407CB7A
 P 5300 4100
-F 0 "C2" H 5350 4200 50  0000 L CNN
+F 0 "C4" H 5350 4200 50  0000 L CNN
 F 1 "0.1u" H 5350 4000 50  0000 L CNN
 	1    5300 4100
@@
 $EndComp
 $Comp
-L CP1 C1
+L CP1 C3
 U 1 1 5407CB6C
 P 4950 4100
-F 0 "C1" H 5000 4200 50  0000 L CNN
+F 0 "C3" H 5000 4200 50  0000 L CNN
 F 1 "100u" H 5000 4000 50  0000 L CNN
 F 2 "E5-10,5_TART" H 4950 4100 60  0001 C CNN
@@
 $EndComp
 $Comp
-L FUSE F1
+L FUSE F2
 U 1 1 5407A432
 P 6100 3600
-F 0 "F1" H 6200 3650 40  0000 C CNN
+F 0 "F2" H 6200 3650 40  0000 C CNN
 F 1 "FUSE" H 6000 3550 40  0000 C CNN
 	1    6100 3600
@@
 $EndComp
 $Comp
-L CP1 C5
+L CP1 C7
 U 1 1 5407A35C
 P 8950 4100
-F 0 "C5" H 9000 4200 50  0000 L CNN
+F 0 "C7" H 9000 4200 50  0000 L CNN
 F 1 "10u" H 9000 4000 50  0000 L CNN
 F 2 "E2-5_TART" H 8950 4100 60  0001 C CNN
@@
 $EndComp
 $Comp
-L C C4
+L C C6
 U 1 1 5407A2F7
 P 7900 4100
-F 0 "C4" H 7950 4200 50  0000 L CNN
+F 0 "C6" H 7950 4200 50  0000 L CNN
 F 1 "0.1u" H 7950 4000 50  0000 L CNN
 	1    7900 4100
@@
 $EndComp
 $Comp
-L CP1 C3
+L CP1 C5
 U 1 1 5407A2C8
 P 7450 4100
-F 0 "C3" H 7500 4200 50  0000 L CNN
+F 0 "C5" H 7500 4200 50  0000 L CNN
 F 1 "10u" H 7500 4000 50  0000 L CNN
 F 2 "E5-10,5_TART" H 7450 4100 60  0001 C CNN
