File: hardware/pcb/kicad/transceiver_block.sch (KiCad schematic (older format))
At the start: 20 parts, among them IC1 LTC2851, IC2 LTC2851, IC3 LTC2851, IC4 LTC2851, IC5 LTC2851, IC6 LTC2851, J1 RJ45, J2 RJ45

Commit message: Getting libraries to work...
Parts:
- removed J1, J2: RJ45, symbol RJ45
- added CON2, CON3: RJ45_TART, symbol RJ45_TART
- renumbered C5 to C10, C1 to C6, C2 to C7, C3 to C8, C4 to C9, IC1 to IC2, IC2 to IC3, IC3 to IC4, IC4 to IC5, IC5 to IC6, IC6 to IC7, R1 to R2, R2 to R3, R3 to R4, R4 to R5, R5 to R6, R6 to R7, R7 to R8
Connections:
- no-connect marks 12 -> 10

Commit message: Routine backup
Parts:
- added C10: 0.1u, symbol C
- renumbered C8 to C11, C9 to C12, C10 to C13, C6 to C8, C7 to C9
Connections:
- net +3V3: now also C10.1
- net GND_A: now also C10.2
