File: hardware/pcb/kicad/transceiver_block.sch (KiCad schematic (older format))
At the start: 21 parts, among them CON2 RJ45_TART, CON3 RJ45_TART, IC2 LTC2851, IC3 LTC2851, IC4 LTC2851, IC5 LTC2851, IC6 LTC2851, IC7 LTC2851

Commit message: Routine backup
Parts:
- added F4: FUSE, ~, symbol FUSE
Connections:
- net +24V: now also F4.2; no longer CON2.1
- new net: CON2.1, F4.1
Changed lines of the file:
@@
 LIBS:valves
 LIBS:TART
+LIBS:spelsberg_box_template_TR
 LIBS:base_station_integrated-cache
 EELAYER 27 0
@@
 $Descr A4 11693 8268
 encoding utf-8
-Sheet 4 7
+Sheet 6 7
 Title ""
-Date "25 sep 2014"
+Date "26 sep 2014"
 Rev ""
 Comp ""
@@
 	2100 1900 2200 1900
 Wire Wire Line
-	2100 7000 2100 1800
+	2100 1800 2100 7000
 Wire Wire Line
 	1700 1700 2200 1700
@@
 	1800 6900 2100 6900
 Wire Wire Line
-	2200 5200 1800 5200
+	1800 5200 2200 5200
 Wire Wire Line
 	1800 5200 1800 5400
 Wire Wire Line
-	2200 4300 1800 4300
+	1800 4300 2200 4300
 Wire Wire Line
 	1800 4300 1800 4500
@@
 	1800 2500 2200 2500
 Wire Wire Line
-	2200 1600 1800 1600
+	1800 1600 2200 1600
 Wire Wire Line
 	1800 1600 1800 1800
@@
 	2200 3500 1700 3500
 Wire Wire Line
-	5050 1050 5050 2800
-Wire Wire Line
 	5050 2800 5200 2800
 Wire Wire Line
@@
 	2100 1800 2200 1800
 Wire Wire Line
-	2200 3400 1800 3400
+	1800 3400 2200 3400
 Wire Wire Line
 	1800 3400 1800 3600
@@
 AR Path="/54092498/5422055D" Ref="C22"  Part="1"
 AR Path="/540670D5/5422055D" Ref="C28"  Part="1"
-F 0 "C16" H 1850 3900 50  0000 L CNN
+F 0 "C28" H 1850 3900 50  0000 L CNN
 F 1 "0.1u" H 1600 3700 50  0000 L CNN
 F 2 "" H 1800 3800 60  0001 C CNN
@@
 AR Path="/54092498/5418D866" Ref="CON7"  Part="1"
 AR Path="/540670D5/5418D866" Ref="CON9"  Part="1"
-F 0 "CON5" H 5850 6550 60  0000 C CNN
+F 0 "CON9" H 5850 6550 60  0000 C CNN
 F 1 "RJ45_TART" H 6250 6600 60  0001 C CNN
 F 2 "" H 5650 6050 60  0001 C CNN
@@
 AR Path="/54092498/5418D832" Ref="CON6"  Part="1"
 AR Path="/540670D5/5418D832" Ref="CON8"  Part="1"
-F 0 "CON4" H 5850 3650 60  0000 C CNN
+F 0 "CON8" H 5850 3650 60  0000 C CNN
 F 1 "RJ45_TART" H 6250 3700 60  0001 C CNN
 F 2 "" H 5650 3150 60  0001 C CNN
@@
 AR Path="/54092498/540678BD" Ref="R16"  Part="1"
 AR Path="/540670D5/540678BD" Ref="R23"  Part="1"
-F 0 "R9" V 4130 1400 50  0000 C CNN
+F 0 "R23" V 4130 1400 50  0000 C CNN
 F 1 "100" V 4050 1400 50  0000 C CNN
 F 2 "" H 4050 1400 60  0001 C CNN
@@
 AR Path="/54092498/540678A5" Ref="R17"  Part="1"
 AR Path="/540670D5/540678A5" Ref="R24"  Part="1"
-F 0 "R10" V 4130 2300 50  0000 C CNN
+F 0 "R24" V 4130 2300 50  0000 C CNN
 F 1 "100" V 4050 2300 50  0000 C CNN
 F 2 "" H 4050 2300 60  0001 C CNN
@@
 AR Path="/54092498/5406788C" Ref="R18"  Part="1"
 AR Path="/540670D5/5406788C" Ref="R25"  Part="1"
-F 0 "R11" V 4130 3200 50  0000 C CNN
+F 0 "R25" V 4130 3200 50  0000 C CNN
 F 1 "100" V 4050 3200 50  0000 C CNN
 F 2 "" H 4050 3200 60  0001 C CNN
@@
 AR Path="/54092498/54067855" Ref="R19"  Part="1"
 AR Path="/540670D5/54067855" Ref="R26"  Part="1"
-F 0 "R12" V 4130 4100 50  0000 C CNN
+F 0 "R26" V 4130 4100 50  0000 C CNN
 F 1 "100" V 4050 4100 50  0000 C CNN
 F 2 "" H 4050 4100 60  0001 C CNN
@@
 AR Path="/54092498/540677FC" Ref="R20"  Part="1"
 AR Path="/540670D5/540677FC" Ref="R27"  Part="1"
-F 0 "R13" V 4130 5000 50  0000 C CNN
+F 0 "R27" V 4130 5000 50  0000 C CNN
 F 1 "100" V 4050 5000 50  0000 C CNN
 F 2 "" H 4050 5000 60  0001 C CNN
@@
 AR Path="/54092498/54067578" Ref="IC19"  Part="1"
 AR Path="/540670D5/54067578" Ref="IC25"  Part="1"
-F 0 "IC13" H 2950 6150 50  0000 C CNN
+F 0 "IC25" H 2950 6150 50  0000 C CNN
 F 1 "LTC2851" H 2950 6350 50  0000 C CNN
 F 2 "MODULE" H 2950 6250 50  0001 C CNN
@@
 AR Path="/54092498/54067576" Ref="IC18"  Part="1"
 AR Path="/540670D5/54067576" Ref="IC24"  Part="1"
-F 0 "IC12" H 2950 5250 50  0000 C CNN
+F 0 "IC24" H 2950 5250 50  0000 C CNN
 F 1 "LTC2851" H 2950 5450 50  0000 C CNN
 F 2 "MODULE" H 2950 5350 50  0001 C CNN
@@
 AR Path="/54092498/54067575" Ref="IC17"  Part="1"
 AR Path="/540670D5/54067575" Ref="IC23"  Part="1"
-F 0 "IC11" H 2950 4350 50  0000 C CNN
+F 0 "IC23" H 2950 4350 50  0000 C CNN
 F 1 "LTC2851" H 2950 4550 50  0000 C CNN
 F 2 "MODULE" H 2950 4450 50  0001 C CNN
@@
 AR Path="/54092498/54067574" Ref="R21"  Part="1"
 AR Path="/540670D5/54067574" Ref="R28"  Part="1"
-F 0 "R14" V 4130 6100 50  0000 C CNN
+F 0 "R28" V 4130 6100 50  0000 C CNN
 F 1 "100" V 4050 6100 50  0000 C CNN
 F 2 "" H 4050 6100 60  0001 C CNN
@@
 AR Path="/54092498/54067573" Ref="R22"  Part="1"
 AR Path="/540670D5/54067573" Ref="R29"  Part="1"
-F 0 "R15" V 4130 6600 50  0000 C CNN
+F 0 "R29" V 4130 6600 50  0000 C CNN
 F 1 "100" V 4050 6600 50  0000 C CNN
 F 2 "" H 4050 6600 60  0001 C CNN
@@
 AR Path="/54092498/54067570" Ref="IC16"  Part="1"
 AR Path="/540670D5/54067570" Ref="IC22"  Part="1"
-F 0 "IC10" H 2950 3450 50  0000 C CNN
+F 0 "IC22" H 2950 3450 50  0000 C CNN
 F 1 "LTC2851" H 2950 3650 50  0000 C CNN
 F 2 "MODULE" H 2950 3550 50  0001 C CNN
@@
 AR Path="/54092498/5406756F" Ref="IC15"  Part="1"
 AR Path="/540670D5/5406756F" Ref="IC21"  Part="1"
-F 0 "IC9" H 2950 2550 50  0000 C CNN
+F 0 "IC21" H 2950 2550 50  0000 C CNN
 F 1 "LTC2851" H 2950 2750 50  0000 C CNN
 F 2 "MODULE" H 2950 2650 50  0001 C CNN
@@
 AR Path="/54092498/5406756E" Ref="IC14"  Part="1"
 AR Path="/540670D5/5406756E" Ref="IC20"  Part="1"
-F 0 "IC8" H 2950 1650 50  0000 C CNN
+F 0 "IC20" H 2950 1650 50  0000 C CNN
 F 1 "LTC2851" H 2950 1850 50  0000 C CNN
 F 2 "MODULE" H 2950 1750 50  0001 C CNN
@@
 AR Path="/54092498/5406756A" Ref="C20"  Part="1"
 AR Path="/540670D5/5406756A" Ref="C26"  Part="1"
-F 0 "C14" H 1850 2100 50  0000 L CNN
+F 0 "C26" H 1850 2100 50  0000 L CNN
 F 1 "0.1u" H 1600 1900 50  0000 L CNN
 F 2 "" H 1800 2000 60  0001 C CNN
@@
 AR Path="/54092498/54067569" Ref="C21"  Part="1"
 AR Path="/540670D5/54067569" Ref="C27"  Part="1"
-F 0 "C15" H 1850 3000 50  0000 L CNN
+F 0 "C27" H 1850 3000 50  0000 L CNN
 F 1 "0.1u" H 1600 2800 50  0000 L CNN
 F 2 "" H 1800 2900 60  0001 C CNN
@@
 AR Path="/54092498/54067568" Ref="C23"  Part="1"
 AR Path="/540670D5/54067568" Ref="C29"  Part="1"
-F 0 "C17" H 1850 4800 50  0000 L CNN
+F 0 "C29" H 1850 4800 50  0000 L CNN
 F 1 "0.1u" H 1600 4600 50  0000 L CNN
 F 2 "" H 1800 4700 60  0001 C CNN
@@
 AR Path="/54092498/54067567" Ref="C24"  Part="1"
 AR Path="/540670D5/54067567" Ref="C30"  Part="1"
-F 0 "C18" H 1850 5700 50  0000 L CNN
+F 0 "C30" H 1850 5700 50  0000 L CNN
 F 1 "0.1u" H 1600 5500 50  0000 L CNN
 F 2 "" H 1800 5600 60  0001 C CNN
@@
 AR Path="/54092498/54067566" Ref="C25"  Part="1"
 AR Path="/540670D5/54067566" Ref="C31"  Part="1"
-F 0 "C19" H 1850 6800 50  0000 L CNN
+F 0 "C31" H 1850 6800 50  0000 L CNN
 F 1 "0.1u" H 1600 6600 50  0000 L CNN
 F 2 "" H 1800 6700 60  0001 C CNN
@@
 	1    0    0    -1
 $EndComp
+$Comp
+L FUSE F4
+U 1 1 54257C9F
+P 5050 1950
+AR Path="/540924B7/54257C9F" Ref="F4"  Part="1"
+AR Path="/54092498/54257C9F" Ref="F5"  Part="1"
+AR Path="/5409247B/54257C9F" Ref="F3"  Part="1"
+AR Path="/540670D5/54257C9F" Ref="F6"  Part="1"
+F 0 "F6" H 5150 2000 40  0000 C CNN
+F 1 "FUSE" H 4950 1900 40  0000 C CNN
+F 2 "~" H 5050 1950 60  0000 C CNN
+F 3 "~" H 5050 1950 60  0000 C CNN
+	1    5050 1950
+	0    -1   -1   0
+$EndComp
+Wire Wire Line
+	5050 2200 5050 2800
+Wire Wire Line
+	5050 1700 5050 1050
 $EndSCHEMATC
