File: hardware/pcb/kicad/radio_hub.sch (KiCad schematic (older format))
At the start: 34 parts

Commit message: Schematic "done" - resolving ERC
Parts:
- removed C? (x2): C, ~, symbol C
- removed C? (x3): CP1, ~, symbol CP1
- removed D?: TVS_DIODE_UNI_TART, ~, symbol TVS_DIODE_UNI_TART
- removed R?: R, ~, symbol R
- removed REG?: OK1-78SR_TART, ~, symbol OK1-78SR_TART
- removed REG?: SPX3940_TART, ~, symbol SPX3940_TART
- removed U?: ACM3225-601-2P-T001_TART, symbol ACM3225-601-2P-T001_TART
- gave numbers to parts that had none: 24
Connections:
- net labels added: _24V_CABLE
- net labels removed: +24V_CABLE, +24v_CABLE
- wire segments 156 -> 101
Other:
- moved on the sheet: LLK, PWR, R15, R7

Commit message: Component values added to schematic. Schematic now passes ERC
Parts:
- added C4, C5, C6, C7: 0.1uF, ~, symbol C
- added IC1: LTC2851_TART, MODULE, symbol LTC2851_TART
- added L1: INDUCTOR, ~, symbol INDUCTOR
- added R13: 100, ~, symbol R
- C2, C3: value C -> 100nF
- C8: value C -> 0.1uF
- R1, R2, R3, R4: value R -> 15k
- R10: value R -> 10k
- R15, R7: value R -> 1k
- R5: value R -> NOT PRESENT
- R6: value R -> 0
- R8: value R -> 82
- R9: value R -> 130
- renumbered L1 to L2, LLK to LLK1, PWR to PWR1
Connections:
- net labels added: +24V_CABLE, +3V3
- net labels removed: +3.3V, CLKIN, PWR, _24V_CABLE
- wire segments 101 -> 145
- no-connect marks 3 -> 5
Other:
- moved on the sheet: L2

Commit message: Added a power switch
Parts:
- R11, R12: value R -> 15k
Changed lines of the file:
@@
 P 7500 5900
 F 0 "R12" V 7580 5900 40  0000 C CNN
-F 1 "R" V 7507 5901 40  0000 C CNN
+F 1 "15k" V 7507 5901 40  0000 C CNN
 F 2 "~" V 7430 5900 30  0000 C CNN
 F 3 "~" H 7500 5900 30  0000 C CNN
@@
 P 7500 6600
 F 0 "R11" V 7580 6600 40  0000 C CNN
-F 1 "R" V 7507 6601 40  0000 C CNN
+F 1 "15k" V 7507 6601 40  0000 C CNN
 F 2 "~" V 7430 6600 30  0000 C CNN
 F 3 "~" H 7500 6600 30  0000 C CNN
@@
 	3900 6450 3700 6450
 Wire Wire Line
-	3700 4250 3700 4850
-Wire Wire Line
-	3700 4850 3700 5150
-Wire Wire Line
-	3700 5150 3700 5550
-Wire Wire Line
-	3700 5550 3700 6450
-Wire Wire Line
-	3700 6450 3700 6650
+	3700 4250 3700 6650
 Wire Wire Line
 	4050 5550 3700 5550
@@
 	5650 4650 5750 4650
 Wire Wire Line
-	5750 4650 5750 4750
-Wire Wire Line
-	5750 4750 5750 5750
-Wire Wire Line
-	5750 5750 5750 5850
-Wire Wire Line
-	5750 5850 5750 6650
+	5750 4650 5750 6650
 Wire Wire Line
 	5650 5750 5750 5750
@@
 	5850 5250 5650 5250
 Wire Wire Line
-	5850 3600 5850 4450
-Wire Wire Line
-	5850 4450 5850 4550
-Wire Wire Line
-	5850 4550 5850 5050
-Wire Wire Line
-	5850 5050 5850 5150
-Wire Wire Line
-	5850 5150 5850 5250
+	5850 3600 5850 5250
 Wire Wire Line
 	5650 5150 5850 5150
@@
 	4050 5650 2850 5650
 Wire Wire Line
-	2350 5550 2350 5650
-Wire Wire Line
-	2350 5650 2350 5750
-Wire Wire Line
-	2000 5650 2350 5650
-Wire Wire Line
-	2350 5650 2450 5650
+	2350 5550 2350 5750
+Wire Wire Line
+	2000 5650 2450 5650
 Connection ~ 2350 5650
 Wire Wire Line
@@
 	7500 5500 7500 5650
 Wire Wire Line
-	7500 6150 7500 6250
-Wire Wire Line
-	7500 6250 7500 6350
+	7500 6150 7500 6350
 Wire Wire Line
 	7500 6850 7500 6950
@@
 	8500 5500 8500 5650
 Wire Wire Line
-	8500 6150 8500 6250
-Wire Wire Line
-	8500 6250 8500 6350
+	8500 6150 8500 6350
 Wire Wire Line
 	8500 6850 8500 6950
@@
 	9400 5500 9400 5650
 Wire Wire Line
-	9400 6150 9400 6250
-Wire Wire Line
-	9400 6250 9400 6350
+	9400 6150 9400 6350
 Wire Wire Line
 	9400 6850 9400 6950
@@
 Connection ~ 9400 6250
 Wire Wire Line
-	10350 6150 10350 6250
-Wire Wire Line
-	10350 6250 10350 6350
+	10350 6150 10350 6350
 Wire Wire Line
 	10350 6850 10350 6950
@@
 	10300 1850 10500 1850
 Wire Wire Line
-	10500 1650 10500 1850
-Wire Wire Line
-	10500 1850 10500 2100
-Wire Wire Line
-	10500 2100 10500 2350
-Wire Wire Line
-	10500 2350 10500 2600
-Wire Wire Line
-	9250 4100 9250 4200
-Wire Wire Line
-	9250 4200 9250 4300
+	10500 1650 10500 2600
+Wire Wire Line
+	9250 4100 9250 4300
 Wire Wire Line
 	9250 4700 9250 4900
@@
 CLK_NINV
 Wire Wire Line
-	6000 1800 6100 1800
-Wire Wire Line
-	6100 1800 6200 1800
-Wire Wire Line
-	6000 1900 6800 1900
-Wire Wire Line
-	6800 1900 6900 1900
+	6000 1800 6200 1800
+Wire Wire Line
+	6000 1900 6900 1900
 $Comp
 L R R13
@@
 	4500 2000 4400 2000
 Wire Wire Line
-	4400 2000 4400 2100
-Wire Wire Line
-	4400 2100 4400 2400
+	4400 2000 4400 2400
 Wire Wire Line
 	4500 2100 4400 2100
@@
 	3500 5050 4050 5050
 Wire Wire Line
-	3500 3600 3500 4550
-Wire Wire Line
-	3500 4550 3500 5050
+	3500 3600 3500 5050
 Wire Wire Line
 	4050 4550 3500 4550
@@
 Connection ~ 10500 1850
 Wire Wire Line
-	10900 1850 10900 2100
-Wire Wire Line
-	10900 2100 10900 2350
-Wire Wire Line
-	10900 2350 10900 2600
+	10900 1850 10900 2600
 Connection ~ 10500 2100
 Connection ~ 10500 2350

Commit message: Address connectivity issues. Removal of connectors and rerouting of tracks
Connections:
- net GND: now also C4.2, C5.2, C6.2, C7.2, LLK1.2 (K); no longer R15.2, R7.2
- net LOL: now also R7.1; no longer LLK1.2 (K)
- net at LLK1.1 (A): now also R7.2; no longer R7.1
- new net GNDINT: R15.2
Other:
- moved on the sheet: LLK1, R7
Changed lines of the file:
@@
 Sheet 1 3
 Title "noname.sch"
-Date "11 nov 2014"
+Date "21 nov 2014"
 Rev ""
 Comp ""
@@
 $EndComp
 $Comp
-L GND #PWR017
-U 1 1 545AA736
-P 7500 4900
-F 0 "#PWR017" H 7500 4900 30  0001 C CNN
-F 1 "GND" H 7500 4830 30  0001 C CNN
-F 2 "" H 7500 4900 60  0000 C CNN
-F 3 "" H 7500 4900 60  0000 C CNN
-	1    7500 4900
-	1    0    0    -1
-$EndComp
-$Comp
 L LED PWR1
 U 1 1 545AA75C
@@
 L R R7
 U 1 1 545AA77F
-P 8500 4550
-F 0 "R7" V 8580 4550 40  0000 C CNN
-F 1 "1k" V 8507 4551 40  0000 C CNN
-F 2 "~" V 8430 4550 30  0000 C CNN
-F 3 "~" H 8500 4550 30  0000 C CNN
-	1    8500 4550
-	1    0    0    -1
-$EndComp
-$Comp
-L GND #PWR018
+P 8500 3950
+F 0 "R7" V 8580 3950 40  0000 C CNN
+F 1 "1k" V 8507 3951 40  0000 C CNN
+F 2 "~" V 8430 3950 30  0000 C CNN
+F 3 "~" H 8500 3950 30  0000 C CNN
+	1    8500 3950
+	1    0    0    -1
+$EndComp
+$Comp
+L GND #PWR017
 U 1 1 545AA78B
 P 8500 4900
-F 0 "#PWR018" H 8500 4900 30  0001 C CNN
+F 0 "#PWR017" H 8500 4900 30  0001 C CNN
 F 1 "GND" H 8500 4830 30  0001 C CNN
 F 2 "" H 8500 4900 60  0000 C CNN
@@
 L LED LLK1
 U 1 1 545AA798
-P 8500 3900
-F 0 "LLK1" H 8500 4000 50  0000 C CNN
-F 1 "LED" H 8500 3800 50  0000 C CNN
-F 2 "~" H 8500 3900 60  0000 C CNN
-F 3 "~" H 8500 3900 60  0000 C CNN
-	1    8500 3900
-	0    -1   -1   0
+P 8500 4600
+F 0 "LLK1" H 8500 4700 50  0000 C CNN
+F 1 "LED" H 8500 4500 50  0000 C CNN
+F 2 "~" H 8500 4600 60  0000 C CNN
+F 3 "~" H 8500 4600 60  0000 C CNN
+	1    8500 4600
+	0    1    1    0
 $EndComp
 Text GLabel 8500 3550 1    60   Input ~ 0
@@
 $EndComp
 $Comp
-L GND #PWR019
+L GND #PWR018
 U 1 1 545ADD26
 P 7500 2900
-F 0 "#PWR019" H 7500 2900 30  0001 C CNN
+F 0 "#PWR018" H 7500 2900 30  0001 C CNN
 F 1 "GND" H 7500 2830 30  0001 C CNN
 F 2 "" H 7500 2900 60  0000 C CNN
@@
 $EndComp
 $Comp
-L VDD #PWR020
+L VDD #PWR019
 U 1 1 545ADEFE
 P 10500 1650
-F 0 "#PWR020" H 10500 1750 30  0001 C CNN
+F 0 "#PWR019" H 10500 1750 30  0001 C CNN
 F 1 "VDD" H 10500 1760 30  0000 C CNN
 F 2 "" H 10500 1650 60  0000 C CNN
@@
 $EndComp
 $Comp
-L VDD #PWR021
+L VDD #PWR020
 U 1 1 545ADF11
 P 9250 3450
-F 0 "#PWR021" H 9250 3550 30  0001 C CNN
+F 0 "#PWR020" H 9250 3550 30  0001 C CNN
 F 1 "VDD" H 9250 3560 30  0000 C CNN
 F 2 "" H 9250 3450 60  0000 C CNN
@@
 $EndComp
 $Comp
-L GND #PWR022
+L GND #PWR021
 U 1 1 545ADF1D
 P 9250 4900
-F 0 "#PWR022" H 9250 4900 30  0001 C CNN
+F 0 "#PWR021" H 9250 4900 30  0001 C CNN
 F 1 "GND" H 9250 4830 30  0001 C CNN
 F 2 "" H 9250 4900 60  0000 C CNN
@@
 Wire Wire Line
 	7500 4100 7500 4300
-Wire Wire Line
-	8500 4100 8500 4300
 $Comp
 L LTC2851_TART IC1
@@
 	4500 1900 4300 1900
 $Comp
-L GND #PWR023
+L GND #PWR022
 U 1 1 54601B73
 P 4400 2400
-F 0 "#PWR023" H 4400 2400 30  0001 C CNN
+F 0 "#PWR022" H 4400 2400 30  0001 C CNN
 F 1 "GND" H 4400 2330 30  0001 C CNN
 F 2 "" H 4400 2400 60  0000 C CNN
@@
 Connection ~ 10500 1850
 Wire Wire Line
-	10900 1850 10900 2600
+	10900 1850 10900 2850
 Connection ~ 10500 2100
 Connection ~ 10500 2350
@@
 $EndComp
 $Comp
-L VDD #PWR024
+L VDD #PWR023
 U 1 1 54629A76
 P 10500 950
-F 0 "#PWR024" H 10500 1050 30  0001 C CNN
+F 0 "#PWR023" H 10500 1050 30  0001 C CNN
 F 1 "VDD" H 10500 1060 30  0000 C CNN
 F 2 "" H 10500 950 60  0000 C CNN
@@
 +3V3
 $Comp
-L PWR_FLAG #FLG025
+L PWR_FLAG #FLG024
 U 1 1 54629A82
 P 10300 1150
-F 0 "#FLG025" H 10300 1245 30  0001 C CNN
+F 0 "#FLG024" H 10300 1245 30  0001 C CNN
 F 1 "PWR_FLAG" H 10300 1330 30  0000 C CNN
 F 2 "" H 10300 1150 60  0000 C CNN
@@
 	1    0    0    -1
 $EndComp
+Wire Wire Line
+	8500 4200 8500 4400
+$Comp
+L GND #PWR025
+U 1 1 54692CDD
+P 10900 2850
+F 0 "#PWR025" H 10900 2850 30  0001 C CNN
+F 1 "GND" H 10900 2780 30  0001 C CNN
+F 2 "" H 10900 2850 60  0000 C CNN
+F 3 "" H 10900 2850 60  0000 C CNN
+	1    10900 2850
+	1    0    0    -1
+$EndComp
+Connection ~ 10900 2600
+Text GLabel 7500 4900 3    60   Input ~ 0
+GNDINT
 $EndSCHEMATC

Commit message: Backup
Parts:
- removed IC2: SI5317, ~, symbol SI5317
- added C1: 0.1uF, ~, symbol C
- added IC2: SI5317_TART, ~, symbol SI5317_TART
Connections:
- net GND is gone; now on net DGND: C2.2, C4.2, C5.2, C6.2, C7.2, C8.2, IC1.3 (DI), IC1.4 (GND), LLK1.2 (K), R1.2, R11.2, R3.2, R5.2, R8.2, SH1.7, X1.2 (GND), X1.4 (GND)
- net +3V3: now also C1.1
- net BWSEL0: now also IC2.22 (BWSEL0)
- net BWSEL1: now also IC2.23 (BWSEL1)
- net CKIN: now also IC2.28 (CLKOUT1+), IC2.29 (CLKOUT1-)
- net DBL2_BY: now also IC2.14 (DBL2_BY)
- net FRQSEL0: now also IC2.24 (FRQSEL0)
- net LOL: now also IC2.18 (LOL)
- net RST: now also IC2.1 (!RST)
- net at C3.2: now also IC2.16 (CKIN+)
- net at C2.1: now also IC2.17 (CKIN-)
- net at X1.1 (X1): now also IC2.6 (XA)
- net at X1.3 (X2): now also IC2.7 (XB)
- net DGND: now reaches SH1.1
- net DGND: now also SH1.10, SH1.11, SH1.12, SH1.2, SH1.3 (GND), SH1.4, SH1.5, SH1.6, SH1.8, SH1.9, C1.2, IC2.11 (RATE0), IC2.15 (RATE1), IC2.19 (DEC), IC2.2 (FRQTBL), IC2.20 (INC), IC2.30 (SFOUT1), IC2.31 (GND), IC2.37 (GND), IC2.8 (GND)
- net VDD renamed VDD_2
- net VDD_2: now also IC2.10 (VDD), IC2.25 (FRQSEL1), IC2.26 (FRQSEL2), IC2.27 (FRQSEL3), IC2.32 (VDD), IC2.33 (SFOUT0), IC2.5 (VDD); no longer L1.2, R2.1, R4.1, R6.1, R9.1
- new net VDD_1: L1.2, R2.1, R4.1, R6.1, R9.1
Other:
- moved on the sheet: C8, LLK1, PWR1, R10, R15, R7, SH1

Commit message: Base station and radio hub boards ready for final checks before manufacture
Changed lines of the file:
@@
 Sheet 1 3
 Title "noname.sch"
-Date "26 nov 2014"
+Date "3 dec 2014"
 Rev ""
 Comp ""
@@
 	3900 6350 3900 6450
 Wire Wire Line
-	3700 6450 3900 6450
+	3900 6450 3700 6450
 Wire Wire Line
 	3700 4250 3700 6650
