File: hardware/pcb/kicad/radios.sch (KiCad schematic (older format))
At the start: 24 parts, among them IC1A LTC2851_TART, IC2A LTC2851_TART, IC3A LTC2851_TART, IC4A LTC2851_TART, IC5A LTC2851_TART, IC6A LTC2851_TART

Commit message: Component values added to schematic. Schematic now passes ERC
Parts:
- CA1, CA2, CA3, CA4, CA5, CA6: value C -> 0.1uF
- RA1, RA2, RA3, RA4, RA5, RA6: value R -> 100
- renumbered IC1A to ICA1, IC2A to ICA2, IC3A to ICA3, IC4A to ICA4, IC5A to ICA5, IC6A to ICA6
Connections:
- net DT_5_INV: now also RA5.2
- net DT_5_NINV: now also RA5.1
- net DT_6_INV: no longer ICA6.5 (Y), RA6.1
- new net DT_6_NINV: ICA6.5 (Y), RA6.1

Commit message: Base station and radio hub boards ready for final checks before manufacture
Parts:
- renumbered MOD_6 to MOD_4, MOD_4 to MOD_6
Changed lines of the file:
@@
 Sheet 3 3
 Title ""
-Date "26 nov 2014"
+Date "3 dec 2014"
 Rev ""
 Comp ""
@@
 $EndComp
 $Comp
-L GPS_RADIO_MODULE_TART MOD_6
+L GPS_RADIO_MODULE_TART MOD_4
 U 1 1 545FFEFE
 P 3500 3900
-F 0 "MOD_6" H 3500 4150 60  0000 C CNN
+F 0 "MOD_4" H 3500 4150 60  0000 C CNN
 F 1 "GPS_RADIO_MODULE_TART" H 3450 3600 60  0001 C CNN
 F 2 "~" H 3500 3900 60  0000 C CNN
@@
 $EndComp
 $Comp
-L GPS_RADIO_MODULE_TART MOD_4
+L GPS_RADIO_MODULE_TART MOD_6
 U 1 1 545FFF0A
 P 3500 5000
-F 0 "MOD_4" H 3500 5250 60  0000 C CNN
+F 0 "MOD_6" H 3500 5250 60  0000 C CNN
 F 1 "GPS_RADIO_MODULE_TART" H 3450 4700 60  0001 C CNN
 F 2 "~" H 3500 5000 60  0000 C CNN
