File: hardware/pcb/radio_hub_module/radio_hub_module.sch (EAGLE design)
At the start: 17 parts, among them CON1 POWER_JACKPTH, IC1 MB16S-TP

Commit message: tidyup. removed outdated schematics. added latest version pcb/schematics
Parts:
- removed C3: 10uF, rcl:CPOL-EUE5-10.5
- removed C4, C5: 0.1uF, rcl:C-EUC0805
- removed CON1: POWER_JACKPTH, SparkFun:POWER_JACKPTH
- removed CON2: (no value), con-lstb:MA03-1
- removed D1: PESD0603-240, texas_lvds:PESD0603-240
- removed F1: SF-1206S050-2, texas_lvds:SF-1206S050-2
- removed R1: 1k, rcl:R-EU_R0603
- removed REG3V3: SPX3940, texas_lvds:SPX3940
- removed REG5V: (no value), texas_lvds:V_REG_OKI-78SRSINK
- added 38.4_MHZ: TSX-3225, texas_lvds:TSX-3225
- added C10, C12, C8: 1u, rcl:C-EUC0603
- added C11, C9: 10n, rcl:C-EUC0603
- added C13, C14, C15, C16: 0.1uF, rcl:C-EUC0402
- added C17, C18: 100nF, rcl:C-EUC0402
- added C19, C21, C24, C26, C27, C28, C29, C30, C31: 0.1u, rcl:C-EUC0805
- added C20: 1uF, rcl:C-EUC0402
- added C22, C23: 100u, rcl:CPOL-EUE5-10.5
- added C25: 10uF, rcl:CPOL-EUE2-5
- added C7: 220u, rcl_1:CPOL-EU1210
- added IC10, IC2, IC3, IC4, IC5, IC6: LTC2851S, texas_lvds:LTC2851S
- added IC11: OKI78s05, texas_lvds:V_REG_OKI-78SRSINK
- added IC12: SPX3940, texas_lvds:SPX3940
- added IC7, IC8: TPS78227DDCR, on_ldo:NCP700BSN
- added IC9: SI5317, texas_lvds:SI5317
- added L1, L2: 220w, wuerth-elektronik:WE-CBF_0805
- added L3: ACM3225-601-2P-T001, texas_lvds:ACM3225-601-2P-T001
- added LLK: Grn, led:LEDCHIPLED_0805
- added MOD_1, MOD_2, MOD_3, MOD_4, MOD_5, MOD_6: GPS_RADIO_MODULE, radio_module:GPS_RADIO_MODULE
- added R10, R9: 0 Ohm, rcl:R-EU_R0805
- added R12: 0 Ohm, resistor:R-EU_R0603
- added R13: Not Present, resistor:R-EU_R0603
- added R14, R15, R21, R22, R25, R26: 15k, resistor:R-EU_R0603
- added R16: 10k, rcl:R-EU_R0402
- added R17, R18: 1k, rcl:R-EU_R0603
- added R19: 130, resistor:R-EU_R0603
- added R20: 82, resistor:R-EU_R0603
- added R23, R27, R28, R29, R30, R31, R32: 100, rcl:R-EU_R0603
- added SH1: BMIS-202, laird:BMIS-202
- added SJ1: (no value), jumper:SJ
- C1: value 100uF -> 1u; device rcl:CPOL-EUE5-10.5 -> rcl:C-EUC0603
- C2: value 10uF -> 220u; device rcl:CPOL-EUE2-5 -> rcl_1:CPOL-EU1210
- CON3, CON4: value (none) -> RJ45-8PTH; device con-lstb:MA03-1 -> SparkFun:RJ45-8PTH
- IC1: value MB16S-TP -> LTC2851S; device texas_lvds:MB16S-TP -> texas_lvds:LTC2851S
- PWR: value (none) -> Red
Connections:
- removed net +24V: C1.+, C4.1, CON2.1, CON4.3, D2.C, F1.2, IC1.+
- removed net GNDINT: C1.-, C2.-, C3.-, C4.2, C5.2, CON2.2, CON2.3, CON3.2, CON4.1, CON4.2, D2.A, IC1.-, PWR.C, REG3V3.GND@2, REG3V3.GND@4, REG5V.GND
- removed net N$2: PWR.A, R1.1
- removed net N$3: F1.1, REG5V.IN
- removed net N$7: CON1.PWR, D1.2, IC1.AC1
- removed net N$8: CON1.GND, D1.1, IC1.AC2
- removed net VCC: C2.+, CON3.1, R1.2, REG3V3.OUT
- new net !DT1: CON3.6, IC1.Z, R27.2
- new net !DT2: CON3.5, IC2.Z, R28.2
- new net !DT3: CON3.2, IC3.Z, R29.2
- new net !DT4: CON4.8, IC4.Z, R30.2
- new net !DT5: CON4.3, IC5.Z, R31.2
- new net !DT6: CON4.4, IC6.Z, R32.2
- new net !RST: C13.2, IC9G$1.!RST, R16.1
- new net +24V_CABLE: CON4.1, L3.1
- new net +2V8_A: C10.1, IC7.OUT, MOD_1.2V8, MOD_2.2V8, MOD_3.2V8
- new net +2V8_B: C12.1, IC8.OUT, MOD_4.2V8, MOD_5.2V8, MOD_6.2V8
- new net +3V3: C1.1, C19.2, C2.+, C25.+, C26.2, C27.2, C28.2, C29.2, C30.2, C31.2, C7.+, C8.1, IC1.VCC, IC10.VCC, IC12.OUT, IC2.VCC, IC3.VCC, IC4.VCC, IC5.VCC, IC6.VCC, IC7.EN, IC7.IN, IC8.EN, IC8.IN, L1.1, L2.1, PWR.C, SJ1.2
- new net 24V_IN: C21.1, C22.+, D2.C, IC11.IN, L3.4
- new net AGND: C10.2, C2.-, C8.2, C9.2, IC7.GND, MOD_1.GND, MOD_2.GND, MOD_3.GND, R9.1
- new net BWSEL0: IC9G$1.BWSEL0, R12.1, R13.2
- new net BWSEL1: IC9G$1.BWSEL1, R14.1, R15.2
- new net BYP: C9.1, IC7.BYP
- new net BYP1: C11.1, IC8.BYP
- new net CKIN: IC9G$1.CKOUT1+, IC9G$1.CKOUT1-, MOD_1.CKIN, MOD_2.CKIN, MOD_3.CKIN, MOD_4.CKIN, MOD_5.CKIN, MOD_6.CKIN
- new net CKIN+: C17.1, IC9G$1.CKIN+
- new net CKIN-: C18.1, IC9G$1.CKIN-
- new net CLK_INV: CON3.7, IC10.A, R23.2
- new net CLK_NINV: CON3.8, IC10.B, R23.1
- new net DBL2_BY: IC9G$1.DBL2_BY, R21.1, R22.2
- new net DT1: CON3.3, IC1.Y, R27.1
- new net DT2: CON3.4, IC2.Y, R28.1
- new net DT3: CON3.1, IC3.Y, R29.1
- new net DT4: CON4.7, IC4.Y, R30.1
- new net DT5: CON4.6, IC5.Y, R31.1
- new net DT6: CON4.5, IC6.Y, R32.1
- new net DT_1: IC1.DI, MOD_1.DT
- new net DT_2: IC2.DI, MOD_2.DT
- new net DT_3: IC3.DI, MOD_3.DT
- new net DT_4: IC4.DI, MOD_4.DT
- new net DT_5: IC5.DI, MOD_5.DT
- new net DT_6: IC6.DI, MOD_6.DT
- new net FRQSEL0: IC9G$1.FRQSEL0, R25.1, R26.2
- new net GND: 38.4_MHZ.GND_1, 38.4_MHZ.GND_2, C13.1, C14.1, C15.1, C16.1, C18.2, C19.1, C20.1, C21.2, C22.-, C23.-, C24.2, C25.-, C26.1, C27.1, C28.1, C29.1, C30.1, C31.1, D2.A, IC1.A, IC1.B, IC1.GND, IC10.DI, IC10.GND, IC11.GND, IC12.GND@2, IC12.GND@4, IC2.A, IC2.B, IC2.GND, IC3.A, IC3.B, IC3.GND, IC4.A, IC4.B, IC4.GND, IC5.A, IC5.B, IC5.GND, IC6.A, IC6.B, IC6.GND, IC9G$1.DEC, IC9G$1.FRQTBL, IC9G$1.GND@8, IC9G$1.GND_@31, IC9G$1.INC, IC9G$1.RATE0, IC9G$1.RATE1, IC9G$1.SFOUT1, L3.3, LLK.A, R10.2, R13.1, R15.1, R17.1, R20.1, R22.1, R26.1, R9.2, SH1.GND@0, SH1.GND@1, SH1.GND@10, SH1.GND@11, SH1.GND@2, SH1.GND@3, SH1.GND@4, SH1.GND@5, SH1.GND@6, SH1.GND@7, SH1.GND@8, SH1.GND@9
- new net GNDA: C1.2, C11.2, C12.2, C7.-, IC8.GND, MOD_4.GND, MOD_5.GND, MOD_6.GND, R10.1
- new net GND_CABLE: CON4.2, L3.2
- new net LOL: IC9G$1.LOL, R18.2
- new net N$1: PWR.A, R17.2
- new net N$11: LLK.C, R18.1
- new net RO_CLK: C17.2, IC10.RO, R19.1, R20.2
- new net VDD: C14.2, C15.2, C16.2, C20.2, IC9G$1.FRQSEL1, IC9G$1.FRQSEL2, IC9G$1.FRQSEL3, IC9G$1.SFOUT0, IC9G$1.VDD_1, IC9G$1.VDD_2, IC9G$1.VDD_3, L2.2, R16.2, R21.2
- new net VDD_2: L1.2, R12.2, R14.2, R19.2, R25.2
- new net XA: 38.4_MHZ.CON_1, IC9G$1.XA
- new net XB: 38.4_MHZ.CON_2, IC9G$1.XB
- net +5V: now also C23.+, C24.1, IC11.OUT, IC12.IN, SJ1.1; no longer C3.+, C5.1, CON3.3, REG3V3.IN, REG5V.OUT
Other:
- note added: "Jumper this when using 3.3V switching Regulator"
