File: hardware/pcb/base201902/base_station_integrated.sch (KiCad schematic (older format))
At the start: 2 parts, among them P1 CONN_20X2, U1 PAPILIO_TART

Commit message: bom update
Parts:
- P1: symbol CONN_20X2 -> base_station_integrated-rescue:CONN_20X2; DIGIKEY (none) -> S9197-ND
- U1: symbol PAPILIO_TART -> TART:PAPILIO_TART
