File: hardware/pcb/base201902/base_station_power_supply.sch (KiCad schematic (older format))
At the start: 19 parts, among them SW1 SWITCH

Commit message: bom update
Parts:
- D1: symbol TVS_DIODE_BI_TART -> TART:TVS_DIODE_BI_TART; DIGIKEY (none) -> PESD0603-240CT-ND
- PC1, PC2, PC3, PC6: symbol CP1 -> base_station_integrated-rescue:CP1
- PC4, PC5, PC7: symbol C -> base_station_integrated-rescue:C
- PCON1: value ~ -> 5.08mm; symbol CONN_2 -> base_station_integrated-rescue:CONN_2; DIGIKEY (none) -> 732-2058-ND; MANUFAC (none) -> + 732-2040-ND
- PD2: value TVS_DIODE_UNI_TART -> 24V UNI TVS; symbol TVS_DIODE_UNI_TART -> TART:TVS_DIODE_UNI_TART; DIGIKEY (none) -> F5823CT-ND
- PF1, PF2: symbol FUSE -> base_station_integrated-rescue:FUSE; DIGIKEY (none) -> 486-1149-1-ND
- PIC1: symbol BRIDGE_TART -> TART:BRIDGE_TART
- PR1: symbol R -> base_station_integrated-rescue:R
- PWR1: symbol LED -> base_station_integrated-rescue:LED
- REG3V3: value SPX3940_TART -> MCP1826; symbol SPX3940_TART -> TART:SPX3940_TART; DIGIKEY (none) -> MCP1826S-3302E/DB-ND; MANUFAC (none) -> MICROCHIP
- REG5V1, REG5V2: symbol OK1-78SR_TART -> TART:OK1-78SR_TART; DIGIKEY (none) -> 811-2196-5-ND
- SW1: symbol SWITCH -> TART:SWITCH; DIGIKEY (none) -> EG2355-ND
