File: hardware/pcb/base201902/transceiver_block.sch (KiCad schematic (older format))
At the start: 25 parts, among them CON5 RJ45_TART, CON6 RJ45_TART, IC13 LTC2851, IC14 LTC2851, IC15 LTC2851, IC16 LTC2851, IC17 LTC2851, IC18 LTC2851

Commit message: bom update
Parts:
- C13, C14, C15, C16, C17, C18, C36, C37, C38: symbol C -> base_station_integrated-rescue:C
- CON5, CON6: symbol RJ45_TART -> TART:RJ45_TART
- F1: value FUSE -> 3.15AF; symbol FUSE -> base_station_integrated-rescue:FUSE; DIGIKEY (none) -> 486-1149-1-ND
- IC13, IC14, IC15, IC16, IC17, IC18: symbol LTC2851 -> base_station_integrated-rescue:LTC2851; DIGIKEY (none) -> LTC2851IS8#PBF-ND
- R15, R16, R17, R18, R19, R20, R21: symbol R -> base_station_integrated-rescue:R
