File: hardware/pcb/hub201902/RadioHub2.1/RadioHub2.1_1.sch (KiCad schematic (older format))
At the start: 55 parts, among them IC13 TPS78227DDCR, IC14 TPS78227DDCR, IC15 TPS78227DDCR, IC7 TPS78227DDCR, IC8 TPS78227DDCR, IC9 TPS78227DDCR

Commit message: bom update
Parts:
- IC13, IC14, IC15, IC7, IC8, IC9: DIGIKEY (none) -> 296-23825-1-ND
- L1, L2, L4, L5, L6, L7: DIGIKEY (none) -> 732-1620-1-ND
- MOD_1, MOD_2, MOD_3, MOD_4, MOD_5, MOD_6, U$1: DIGIKEY (none) -> N/A
Changed lines of the file:
@@
 F 2 "RadioHub2.1:SOT23-5" H 3100 1300 50  0001 C CNN
 F 3 "" H 3100 1300 50  0001 C CNN
+F 4 "296-23825-1-ND" H 0   0   50  0001 C CNN "DIGIKEY"
 	1    3100 1300
 	1    0    0    -1
@@
 F 2 "RadioHub2.1:GPS_RADIO_MODULE" H 4800 1200 50  0001 C CNN
 F 3 "" H 4800 1200 50  0001 C CNN
+F 4 "N/A" H 0   0   50  0001 C CNN "DIGIKEY"
 	1    4800 1200
 	1    0    0    -1
@@
 F 2 "RadioHub2.1:GPS_RADIO_MODULE" H 4800 3100 50  0001 C CNN
 F 3 "" H 4800 3100 50  0001 C CNN
+F 4 "N/A" H 0   0   50  0001 C CNN "DIGIKEY"
 	1    4800 3100
 	1    0    0    -1
@@
 F 2 "RadioHub2.1:GPS_RADIO_MODULE" H 4800 4900 50  0001 C CNN
 F 3 "" H 4800 4900 50  0001 C CNN
+F 4 "N/A" H 0   0   50  0001 C CNN "DIGIKEY"
 	1    4800 4900
 	1    0    0    -1
@@
 F 2 "RadioHub2.1:GPS_RADIO_MODULE" H 9800 1200 50  0001 C CNN
 F 3 "" H 9800 1200 50  0001 C CNN
+F 4 "N/A" H 0   0   50  0001 C CNN "DIGIKEY"
 	1    9800 1200
 	1    0    0    -1
@@
 F 2 "RadioHub2.1:GPS_RADIO_MODULE" H 9800 3100 50  0001 C CNN
 F 3 "" H 9800 3100 50  0001 C CNN
+F 4 "N/A" H 0   0   50  0001 C CNN "DIGIKEY"
 	1    9800 3100
 	1    0    0    -1
@@
 F 2 "RadioHub2.1:GPS_RADIO_MODULE" H 9800 4900 50  0001 C CNN
 F 3 "" H 9800 4900 50  0001 C CNN
+F 4 "N/A" H 0   0   50  0001 C CNN "DIGIKEY"
 	1    9800 4900
 	1    0    0    -1
@@
 F 2 "RadioHub2.1:SOT23-5" H 3100 3200 50  0001 C CNN
 F 3 "" H 3100 3200 50  0001 C CNN
+F 4 "296-23825-1-ND" H 0   0   50  0001 C CNN "DIGIKEY"
 	1    3100 3200
 	1    0    0    -1
@@
 F 2 "RadioHub2.1:0805" H 1600 1200 50  0001 C CNN
 F 3 "" H 1600 1200 50  0001 C CNN
+F 4 "732-1620-1-ND" H 0   0   50  0001 C CNN "DIGIKEY"
 	1    1600 1200
 	1    0    0    -1
@@
 F 2 "RadioHub2.1:0805" H 1600 3100 50  0001 C CNN
 F 3 "" H 1600 3100 50  0001 C CNN
+F 4 "732-1620-1-ND" H 0   0   50  0001 C CNN "DIGIKEY"
 	1    1600 3100
 	1    0    0    -1
@@
 F 2 "RadioHub2.1:SOT23-5" H 3100 5000 50  0001 C CNN
 F 3 "" H 3100 5000 50  0001 C CNN
+F 4 "296-23825-1-ND" H 0   0   50  0001 C CNN "DIGIKEY"
 	1    3100 5000
 	1    0    0    -1
@@
 F 2 "RadioHub2.1:0805" H 1600 4900 50  0001 C CNN
 F 3 "" H 1600 4900 50  0001 C CNN
+F 4 "732-1620-1-ND" H 0   0   50  0001 C CNN "DIGIKEY"
 	1    1600 4900
 	1    0    0    -1
@@
 F 2 "RadioHub2.1:SOT23-5" H 8100 1300 50  0001 C CNN
 F 3 "" H 8100 1300 50  0001 C CNN
+F 4 "296-23825-1-ND" H 0   0   50  0001 C CNN "DIGIKEY"
 	1    8100 1300
 	1    0    0    -1
@@
 F 2 "RadioHub2.1:SOT23-5" H 8100 3200 50  0001 C CNN
 F 3 "" H 8100 3200 50  0001 C CNN
+F 4 "296-23825-1-ND" H 0   0   50  0001 C CNN "DIGIKEY"
 	1    8100 3200
 	1    0    0    -1
@@
 F 2 "RadioHub2.1:0805" H 6600 1200 50  0001 C CNN
 F 3 "" H 6600 1200 50  0001 C CNN
+F 4 "732-1620-1-ND" H 0   0   50  0001 C CNN "DIGIKEY"
 	1    6600 1200
 	1    0    0    -1
@@
 F 2 "RadioHub2.1:0805" H 6600 3100 50  0001 C CNN
 F 3 "" H 6600 3100 50  0001 C CNN
+F 4 "732-1620-1-ND" H 0   0   50  0001 C CNN "DIGIKEY"
 	1    6600 3100
 	1    0    0    -1
@@
 F 2 "RadioHub2.1:SOT23-5" H 8100 5000 50  0001 C CNN
 F 3 "" H 8100 5000 50  0001 C CNN
+F 4 "296-23825-1-ND" H 0   0   50  0001 C CNN "DIGIKEY"
 	1    8100 5000
 	1    0    0    -1
@@
 F 2 "RadioHub2.1:0805" H 6600 4900 50  0001 C CNN
 F 3 "" H 6600 4900 50  0001 C CNN
+F 4 "732-1620-1-ND" H 0   0   50  0001 C CNN "DIGIKEY"
 	1    6600 4900
 	1    0    0    -1
@@
 F 2 "RadioHub2.1:LOGO" H 1400 6900 50  0001 C CNN
 F 3 "" H 1400 6900 50  0001 C CNN
+F 4 "N/A" H 0   0   50  0001 C CNN "DIGIKEY"
 	1    1400 6900
 	1    0    0    -1
