File: hardware/pcb/hub201902/RadioHub2.1/RadioHub2.1_2.sch (KiCad schematic (older format))
At the start: 20 parts, among them CON3 RJ45-8PTH, CON4 RJ45-8PTH, IC11 OKI78s05, IC12 SPX3940, U1 MAX3284E

Commit message: bom update
Parts:
- 24V, 24VF, 3V3, 5V: DIGIKEY (none) -> N/A
- CON3, CON4: DIGIKEY (none) -> 609-1046-ND; Notes (none) -> Almost any 8p8c will do
- D2: value SMF24A -> UNI 24V TVS; DIGIKEY (none) -> F5823CT-ND
- IC11: DIGIKEY (none) -> 811-2196-5-ND
- IC12: DIGIKEY (none) -> MCP1826S-3302E/DB-ND
- L3: value ACM3225-601-2P-T001 -> ACP3225-102-2P-TL000; DIGIKEY (none) -> 445-174210-1-ND
- U1: DIGIKEY (none) -> MAX3284EAUT+CT-ND
Changed lines of the file:
@@
 F 2 "RadioHub2.1:RJ45-8" H 3400 1600 50  0001 C CNN
 F 3 "" H 3400 1600 50  0001 C CNN
+F 4 "609-1046-ND" H 0   0   50  0001 C CNN "DIGIKEY"
+F 5 "Almost any 8p8c will do " H 0   0   50  0001 C CNN "Notes"
 	1    3400 1600
 	-1   0    0    1
@@
 AR Path="/5C5BA189/FA53E63416675DB9" Ref="L3"  Part="1"
 F 0 "L3" H 6600 1200 50  0001 C CNN
-F 1 "ACM3225-601-2P-T001" H 6600 1200 50  0001 C CNN
+F 1 "ACP3225-102-2P-TL000" H 6600 1200 50  0001 C CNN
 F 2 "RadioHub2.1:ACM3225-601-2P-T001" H 6600 1200 50  0001 C CNN
 F 3 "" H 6600 1200 50  0001 C CNN
+F 4 "445-174210-1-ND" H 0   0   50  0001 C CNN "DIGIKEY"
 	1    6600 1200
 	1    0    0    -1
@@
 F 2 "RadioHub2.1:TO220-IGO" H 8700 1000 50  0001 C CNN
 F 3 "" H 8700 1000 50  0001 C CNN
+F 4 "811-2196-5-ND" H 0   0   50  0001 C CNN "DIGIKEY"
 	1    8700 1000
 	1    0    0    -1
@@
 AR Path="/5C5BA189/4C475A1A20478EC3" Ref="D2"  Part="1"
 F 0 "D2" H 8110 1275 59  0000 L BNN
-F 1 "SMF24A" H 7960 1045 59  0000 L BNN
+F 1 "UNI 24V TVS" H 7960 1045 59  0000 L BNN
 F 2 "RadioHub2.1:SOD123" H 8200 1200 50  0001 C CNN
 F 3 "" H 8200 1200 50  0001 C CNN
+F 4 "F5823CT-ND" H 0   0   50  0001 C CNN "DIGIKEY"
 	1    8200 1200
 	0    -1   -1   0
@@
 F 2 "RadioHub2.1:SOT223" H 8700 3700 50  0001 C CNN
 F 3 "" H 8700 3700 50  0001 C CNN
+F 4 "MCP1826S-3302E/DB-ND" H 0   0   50  0001 C CNN "DIGIKEY"
 	1    8700 3700
 	1    0    0    -1
@@
 F 2 "RadioHub2.1:RJ45-8" H 1700 1600 50  0001 C CNN
 F 3 "" H 1700 1600 50  0001 C CNN
+F 4 "609-1046-ND" H 0   0   50  0001 C CNN "DIGIKEY"
+F 5 "Almost any 8p8c will do " H 0   0   50  0001 C CNN "Notes"
 	1    1700 1600
 	-1   0    0    1
@@
 F 2 "RadioHub2.1:SOT23-6L" H 5700 3600 50  0001 C CNN
 F 3 "" H 5700 3600 50  0001 C CNN
+F 4 "MAX3284EAUT+CT-ND" H 0   0   50  0001 C CNN "DIGIKEY"
 	1    5700 3600
 	-1   0    0    1
@@
 F 2 "RadioHub2.1:TP20SQ" H 6100 900 50  0001 C CNN
 F 3 "" H 6100 900 50  0001 C CNN
+F 4 "N/A" H 0   0   50  0001 C CNN "DIGIKEY"
 	1    6100 900
 	-1   0    0    1
@@
 F 2 "RadioHub2.1:TP20SQ" H 10300 900 50  0001 C CNN
 F 3 "" H 10300 900 50  0001 C CNN
+F 4 "N/A" H 0   0   50  0001 C CNN "DIGIKEY"
 	1    10300 900
 	-1   0    0    1
@@
 F 2 "RadioHub2.1:TP20SQ" H 9500 3000 50  0001 C CNN
 F 3 "" H 9500 3000 50  0001 C CNN
+F 4 "N/A" H 0   0   50  0001 C CNN "DIGIKEY"
 	1    9500 3000
 	-1   0    0    1
@@
 F 2 "RadioHub2.1:TP20SQ" H 7400 900 50  0001 C CNN
 F 3 "" H 7400 900 50  0001 C CNN
+F 4 "N/A" H 0   0   50  0001 C CNN "DIGIKEY"
 	1    7400 900
 	-1   0    0    1
