File: hardware/pcb/hub201902/RadioHub2.1/RadioHub2.1_3.sch (KiCad schematic (older format))
At the start: 24 parts, among them U2 MAX3295AUT, U3 MAX3295AUT, U4 MAX3295AUT, U5 MAX3295AUT, U6 MAX3295AUT, U7 MAX3295AUT

Commit message: bom update
Parts:
- U2, U3, U4, U5, U6, U7: DIGIKEY (none) -> ISL3295EIHZ-TCT-ND
Changed lines of the file:
@@
 F 2 "RadioHub2.1:SOT23-6L" H 2800 1400 50  0001 C CNN
 F 3 "" H 2800 1400 50  0001 C CNN
+F 4 "ISL3295EIHZ-TCT-ND" H 0   0   50  0001 C CNN "DIGIKEY"
 	1    2800 1400
 	-1   0    0    -1
@@
 F 2 "RadioHub2.1:SOT23-6L" H 6100 1400 50  0001 C CNN
 F 3 "" H 6100 1400 50  0001 C CNN
+F 4 "ISL3295EIHZ-TCT-ND" H 0   0   50  0001 C CNN "DIGIKEY"
 	1    6100 1400
 	-1   0    0    -1
@@
 F 2 "RadioHub2.1:SOT23-6L" H 9400 1400 50  0001 C CNN
 F 3 "" H 9400 1400 50  0001 C CNN
+F 4 "ISL3295EIHZ-TCT-ND" H 0   0   50  0001 C CNN "DIGIKEY"
 	1    9400 1400
 	-1   0    0    -1
@@
 F 2 "RadioHub2.1:SOT23-6L" H 2800 4400 50  0001 C CNN
 F 3 "" H 2800 4400 50  0001 C CNN
+F 4 "ISL3295EIHZ-TCT-ND" H 0   0   50  0001 C CNN "DIGIKEY"
 	1    2800 4400
 	-1   0    0    -1
@@
 F 2 "RadioHub2.1:SOT23-6L" H 6100 4400 50  0001 C CNN
 F 3 "" H 6100 4400 50  0001 C CNN
+F 4 "ISL3295EIHZ-TCT-ND" H 0   0   50  0001 C CNN "DIGIKEY"
 	1    6100 4400
 	-1   0    0    -1
@@
 F 2 "RadioHub2.1:SOT23-6L" H 9400 4400 50  0001 C CNN
 F 3 "" H 9400 4400 50  0001 C CNN
+F 4 "ISL3295EIHZ-TCT-ND" H 0   0   50  0001 C CNN "DIGIKEY"
 	1    9400 4400
 	-1   0    0    -1
