File: hardware/pcb/hub201902/RadioHub2.1/RadioHub2.1_4.sch (KiCad schematic (older format))
At the start: 23 parts, among them U8 CDCLVC1106

Commit message: bom update
Parts:
- U8: DIGIKEY (none) -> 296-27588-1-ND
Changed lines of the file:
@@
 F 2 "RadioHub2.1:SSOP14" H 5900 2300 50  0001 C CNN
 F 3 "" H 5900 2300 50  0001 C CNN
+F 4 "296-27588-1-ND" H 0   0   50  0001 C CNN "DIGIKEY"
 	1    5900 2300
 	1    0    0    -1
