File: hardware/pcb/front_end_block201902/front_end_block.sch (KiCad schematic (older format))
At the start: 29 parts, among them T1 DDTC114, T2 DDTC114, U1 MAX2769LPKF, X1 SMA

Commit message: Added BOM stuff
Parts:
- T1, T2: DIGIKEY (none) -> DTC114YET1GOSCT-ND
- U1: DIGIKEY (none) -> 700-MAX2769CETI+; Notes (none) -> Mouser
- X1: DIGIKEY (none) -> CON-SMA-EDGE-S-ND; Notes (none) -> Normally bulk sourced
Changed lines of the file:
@@
 F 2 "front_end_block:QFN28LPKF" H 4700 4800 50  0001 C CNN
 F 3 "" H 4700 4800 50  0001 C CNN
+F 4 "700-MAX2769CETI+" H 0   0   50  0001 C CNN "DIGIKEY"
+F 5 "Mouser" H 0   0   50  0001 C CNN "Notes"
 	1    4700 4800
 	1    0    0    -1
@@
 F 2 "front_end_block:J502-ND-142-0701-801_806" H 2700 3400 50  0001 C CNN
 F 3 "" H 2700 3400 50  0001 C CNN
+F 4 "CON-SMA-EDGE-S-ND" H 0   0   50  0001 C CNN "DIGIKEY"
+F 5 "Normally bulk sourced" H 0   0   50  0001 C CNN "Notes"
 	1    2700 3400
 	1    0    0    -1
@@
 F 2 "front_end_block:J502-ND-142-0701-801_806" H 9400 4300 50  0001 C CNN
 F 3 "" H 9400 4300 50  0001 C CNN
+F 4 "CON-SMA-EDGE-S-ND" H 0   0   50  0001 C CNN "DIGIKEY"
+F 5 "Normally bulk sourced" H 0   0   50  0001 C CNN "Notes"
 	2    9400 4300
 	-1   0    0    -1
@@
 F 2 "front_end_block:SOT323-R_INFINEON" H 7800 2900 50  0001 C CNN
 F 3 "" H 7800 2900 50  0001 C CNN
+F 4 "DTC114YET1GOSCT-ND" H 0   0   50  0001 C CNN "DIGIKEY"
 	1    7800 2900
 	-1   0    0    -1
@@
 F 2 "front_end_block:SOT323-R_INFINEON" H 6400 3000 50  0001 C CNN
 F 3 "" H 6400 3000 50  0001 C CNN
+F 4 "DTC114YET1GOSCT-ND" H 0   0   50  0001 C CNN "DIGIKEY"
 	1    6400 3000
 	-1   0    0    -1
