File: hardware/pcb/base_station/base_station_clock.sch (KiCad schematic (older format))
At the start: 8 parts, among them IC26 XTAL_DRIVER_TART, X1 TCXO_TART

Commit message: Moved things around so that old files are in the legacy directory
Parts:
- added U2: BMIS-105_BMIS-205, ~, symbol BMIS-105_BMIS-205
- C25, C26, R29, R30, R31, R32: footprint (none) -> SM0603
- IC26: footprint MODULE -> 6TSSOP_TART
- X1: footprint MODULE -> 4_SMD_TART
Connections:
- net GND: now also U2.1, U2.10, U2.11, U2.12, U2.13, U2.14, U2.15, U2.16, U2.17, U2.18, U2.19, U2.2, U2.20, U2.21, U2.22, U2.23, U2.24, U2.3 (GND), U2.4, U2.5, U2.6, U2.7, U2.8, U2.9
Changed lines of the file:
@@
 Sheet 7 7
 Title ""
-Date "8 dec 2014"
+Date "13 feb 2015"
 Rev ""
 Comp ""
@@
 F 0 "IC26" H 7050 3670 50  0000 C CNN
 F 1 "XTAL_DRIVER_TART" H 7050 4030 50  0001 C CNN
-F 2 "MODULE" H 7070 3190 50  0001 C CNN
+F 2 "6TSSOP_TART" H 7070 3190 50  0000 C CNN
 F 3 "DOCUMENTATION" H 7050 3270 50  0001 C CNN
 F 4 "XTAL_DRIVER" H 7060 3860 50  0000 C CNN "NAME"
@@
 F 0 "X1" H 4200 3550 50  0000 C CNN
 F 1 "TCXO_TART" H 4210 4190 50  0001 C CNN
-F 2 "MODULE" H 4190 4010 50  0001 C CNN
+F 2 "4_SMD_TART" H 4190 4010 50  0000 C CNN
 F 3 "DOCUMENTATION" H 4200 4100 50  0001 C CNN
 F 4 "TCXO" H 4190 3750 50  0000 C CNN "NAME"
@@
 	6100 3650 6100 3950
 Wire Wire Line
-	6300 3750 5650 3750
+	5650 3750 6300 3750
 Wire Wire Line
 	4950 3750 5250 3750
@@
 	7800 3650 8000 3650
 Wire Wire Line
-	8000 4000 8000 3300
+	8000 3300 8000 4000
 Connection ~ 8000 3650
 Wire Wire Line
-	5850 3950 5850 3300
+	5850 3300 5850 3950
 Wire Wire Line
 	7800 3750 8300 3750
@@
 F 0 "C25" H 8050 4300 50  0000 L CNN
 F 1 "0.1u" H 8050 4100 50  0000 L CNN
-F 2 "" H 8000 4200 60  0001 C CNN
+F 2 "SM0603" H 8000 4200 60  0000 C CNN
 F 3 "" H 8000 4200 60  0001 C CNN
 	1    8000 4200
@@
 F 0 "R29" V 8080 3050 50  0000 C CNN
 F 1 "0" V 8000 3050 50  0000 C CNN
-F 2 "" H 8000 3050 60  0001 C CNN
+F 2 "SM0603" H 8000 3050 60  0000 C CNN
 F 3 "" H 8000 3050 60  0001 C CNN
 	1    8000 3050
@@
 F 0 "R30" V 6180 4200 50  0000 C CNN
 F 1 "0" V 6100 4200 50  0000 C CNN
-F 2 "" H 6100 4200 60  0001 C CNN
+F 2 "SM0603" H 6100 4200 60  0000 C CNN
 F 3 "" H 6100 4200 60  0001 C CNN
 	1    6100 4200
@@
 F 0 "R31" V 5930 4200 50  0000 C CNN
 F 1 "10k" V 5850 4200 50  0000 C CNN
-F 2 "" H 5850 4200 60  0001 C CNN
+F 2 "SM0603" H 5850 4200 60  0000 C CNN
 F 3 "" H 5850 4200 60  0001 C CNN
 	1    5850 4200
@@
 F 0 "R32" V 5930 3050 50  0000 C CNN
 F 1 "10k" V 5850 3050 50  0000 C CNN
-F 2 "" H 5850 3050 60  0001 C CNN
+F 2 "SM0603" H 5850 3050 60  0000 C CNN
 F 3 "" H 5850 3050 60  0001 C CNN
 	1    5850 3050
@@
 F 0 "C26" H 5500 3850 50  0000 L CNN
 F 1 "2200p" H 5500 3650 50  0000 L CNN
-F 2 "" H 5450 3750 60  0001 C CNN
+F 2 "SM0603" H 5450 3750 60  0000 C CNN
 F 3 "" H 5450 3750 60  0001 C CNN
 	1    5450 3750
 	0    -1   -1   0
 $EndComp
+$Comp
+L GND #PWR016
+U 1 1 54DD2F01
+P 5450 5750
+F 0 "#PWR016" H 5450 5750 30  0001 C CNN
+F 1 "GND" H 5450 5680 30  0001 C CNN
+F 2 "" H 5450 5750 60  0001 C CNN
+F 3 "" H 5450 5750 60  0001 C CNN
+	1    5450 5750
+	1    0    0    -1
+$EndComp
+Wire Wire Line
+	4950 5550 4950 5650
+Wire Wire Line
+	4950 5650 6100 5650
+Wire Wire Line
+	5900 5650 5900 5550
+Wire Wire Line
+	5450 5550 5450 5750
+Connection ~ 5450 5650
+Wire Wire Line
+	5000 5550 5000 5650
+Connection ~ 5000 5650
+Wire Wire Line
+	5050 5550 5050 5650
+Connection ~ 5050 5650
+Wire Wire Line
+	5100 5550 5100 5650
+Connection ~ 5100 5650
+Wire Wire Line
+	5150 5550 5150 5650
+Connection ~ 5150 5650
+Wire Wire Line
+	5200 5550 5200 5650
+Connection ~ 5200 5650
+Wire Wire Line
+	5250 5550 5250 5650
+Connection ~ 5250 5650
+Wire Wire Line
+	5300 5550 5300 5650
+Connection ~ 5300 5650
+Wire Wire Line
+	5350 5550 5350 5650
+Connection ~ 5350 5650
+Wire Wire Line
+	5400 5550 5400 5650
+Connection ~ 5400 5650
+Wire Wire Line
+	5500 5550 5500 5650
+Connection ~ 5500 5650
+Wire Wire Line
+	5550 5550 5550 5650
+Connection ~ 5550 5650
+Wire Wire Line
+	5600 5550 5600 5650
+Connection ~ 5600 5650
+Wire Wire Line
+	5650 5550 5650 5650
+Connection ~ 5650 5650
+Wire Wire Line
+	5700 5550 5700 5650
+Connection ~ 5700 5650
+Wire Wire Line
+	5750 5550 5750 5650
+Connection ~ 5750 5650
+Wire Wire Line
+	5800 5550 5800 5650
+Connection ~ 5800 5650
+Wire Wire Line
+	5850 5550 5850 5650
+Connection ~ 5850 5650
+$Comp
+L BMIS-105_BMIS-205 U2
+U 1 1 54DF59A6
+P 5450 5350
+F 0 "U2" H 5550 5250 0   0001 C CNN
+F 1 "BMIS-105_BMIS-205" H 5550 5250 0   0001 C CNN
+F 2 "~" H 5550 5250 60  0000 C CNN
+F 3 "~" H 5550 5250 60  0000 C CNN
+	1    5450 5350
+	1    0    0    -1
+$EndComp
+Wire Wire Line
+	5950 5650 5950 5550
+Connection ~ 5900 5650
+Wire Wire Line
+	6000 5650 6000 5550
+Connection ~ 5950 5650
+Wire Wire Line
+	6050 5650 6050 5550
+Connection ~ 6000 5650
+Wire Wire Line
+	6100 5650 6100 5550
+Connection ~ 6050 5650
 $EndSCHEMATC
