File: hardware/pcb/base_station/base_station_integrated.sch (KiCad schematic (older format))
At the start: 2 parts, among them P1 CONN_20X2, U1 PAPILIO_TART

Commit message: Moved things around so that old files are in the legacy directory
Parts:
- P1: footprint (none) -> RASP_PI_B+_TART
- U1: footprint (none) -> PAPILIO_TART
Connections:
- net +5V: now also U1.AH11 (+5V), U1.AL3 (+5V), U1.BH11 (+5V), U1.CH11 (+5V), U1.CL3 (+5V); no longer U1.AH8 (GND)
- net CLK_OUT_1: no longer U1.C15
- net CLK_OUT_2: no longer U1.B7
- net CLK_OUT_3: no longer U1.B3
- net CLK_OUT_4: no longer U1.C3
- net GND: now also U1.AH8 (GND), U1.AL0 (GND); no longer U1.AH11 (+5V), U1.AL3 (+5V)
- net START: no longer U1.B8
- no-connect marks 46 -> 57
