File: hardware/pcb/legacy/base_station/base_station_integrated.sch (KiCad schematic (older format))
At the start: 2 parts, among them P1 CONN_20X2, U1 PAPILIO_TART

Commit message: Moved things around so that old files are in the legacy directory
Parts:
- P1: footprint RASP_PI_B+_TART -> (none)
- U1: footprint PAPILIO_TART -> (none)
Connections:
- net +5V: now also U1.5A8 (+5V); no longer U1.5B11 (+5V0), U1.5C11 (+5V0), U1.5C3 (+5V0), U1.GA11 (GND), U1.GC8 (GND)
- net CLK_OUT_1: now also U1.C15
- net CLK_OUT_2: now also U1.B7
- net CLK_OUT_3: now also U1.B3
- net CLK_OUT_4: now also U1.C3
- net GND: now also U1.GA11 (GND); no longer U1.5A8 (+5V), U1.5C11 (+5V0)
- net START: now also U1.B8
- no-connect marks 57 -> 46
